File: power-wedge-control.sch (KiCad schematic (older format))
At the start: 15 parts, among them J1 Conn_01x02, J2 Conn_01x03, J3 Conn_01x02, Q1 MMBT3904L, Q2 DMP3099L, Q3 MMBT3904L, Q4 DMP3099L

Commit message: KiCad 6. Add 7805 reg, Arduino Uno, ESP32 footprints, angle sensor input
Add todo notes.
WIP.
Parts:
- added C1, C2: 470n, Capacitor_SMD:C_0603_1608Metric, symbol Device:C
- added C3, C4: NOSTUFF, Capacitor_SMD:C_0603_1608Metric, symbol Device:C
- added J4, J5: Conn_01x03, TerminalBlock_Phoenix:TerminalBlock_Phoenix_PT-1,5-3-3.5-H_1x03_P3.50mm_Horizontal, symbol Connector_Generic:Conn_01x03
- added L1, L2: 600R/200mA, Inductor_SMD:L_0603_1608Metric, symbol Device:L
- added R7, R8: 200k, Resistor_SMD:R_0603_1608Metric, symbol Device:R
Connections:
- net labels added: ANGL1, ANGL2, SENS_PWR
- wire segments 26 -> 48
Other:
- note added: "Display design:\n 7-segment w/ dot for moving?\n 2 displays: 1 for set point, 1 for actual?\n 3 small digits for angle, 1 large for set point?\n Use hex so angle fits in one digit.\n LCD?\n OLED?"
- note added: "Relay Control"
- note added: "TODO: 5V buck power supply from 12V"
- note added: "TODO: Analog front end?"
- note added: "TODO: HW switch pin to disable control inside MCU?"
- note added: "TODO: HW switch to disconnect relays from MCU?"
- note added: "TODO: Indicator LEDs for relays."
- note added: "TODO: Load switch controlling sensor power (for turn on slew rate or sleep)?"
- note added: "TODO: Manual control option? External relay enable? Or just from MCU?"
- note added: "TODO: Optocouplers on relay enable pins to isolate MCU from 12V?"
- note added: "TODO: Reverse polarity, short-circuit, power good?"
- note added: "TODO: When to sleep/power down?\n A: 1.) Stay ON anytime that the wedge is DOWN.\n 2.) Turn ON for 30 secs after a button press (if wedge is not down)."
- note added: "To Angle Sensor 1"
- note added: "To Angle Sensor 2"
- moved on the sheet: D1, D2, J2, Q1, Q2, Q3, Q4, R1, R2, R3, R4, R5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
