File: hw-debounce.kicad_sch (KiCad schematic)
At the start: 13 parts, among them U2 NC7WZ14P6X

Commit message: Fix hardware debounce circuit (was incorrect).
Connections:
- net SW1IN: no longer U2.1 (A1)
- net SW2IN: no longer U2.3 (A2)
- net at C11.1, C12.1, D4.1 (K)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: now also U2.3 (A2)
- net at C10.1, C9.1, D3.1 (K)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: now also U2.1 (A1)
Other:
- moved on the sheet: C10, C11, C12, C9, D3, D4, R15, R16, R17, R18, R19, R20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
