File: hw-debounce.kicad_sch (KiCad schematic)
At the start: 13 parts, among them U2 NC7WZ14P6X

Commit message: WIP. Add support for active-high (15V max) switch input to schematic.
Connections:
- net SW1IN renamed ~{SW1IN}
- net SW2IN renamed ~{SW2IN}
Other:
- note added: "Expecting GND or open on switch inputs."
Changed lines of the file:
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@@
     (stroke (width 0) (type default) (color 0 0 0 0))
+  )
+  (text "Expecting GND or open on switch inputs." (at 73.66 118.11 0)
+    (effects (font (size 1.27 1.27)) (justify left bottom))
   )
   (text "External Switch\nContacts" (at 91.44 99.06 180)
@@
     (effects (font (size 1.524 1.524)) (justify left))
   )
-  (hierarchical_label "SW2IN" (shape bidirectional) (at 127 101.6 180)
+  (hierarchical_label "~{SW2IN}" (shape bidirectional) (at 127 101.6 180)
     (effects (font (size 1.27 1.27)) (justify right))
   )
@@
     (effects (font (size 1.524 1.524)) (justify right))
   )
-  (hierarchical_label "SW1IN" (shape bidirectional) (at 91.44 87.63 180)
+  (hierarchical_label "~{SW1IN}" (shape bidirectional) (at 91.44 87.63 180)
     (effects (font (size 1.27 1.27)) (justify right))
   )
