File: power-wedge-control.kicad_pcb (KiCad board)
At the start: 2 copper layers, 28.4 x 41.4 mm, 15 parts, among them J1 Conn_01x02, J2 Conn_01x03, J3 Conn_01x02, Q1 MMBT3904L, Q2 DMP3099L, Q3 MMBT3904L, Q4 DMP3099L

Commit message: KiCad 6. Add 7805 reg, Arduino Uno, ESP32 footprints, angle sensor input
Add todo notes.
WIP.
Parts:
- added A1: Arduino_UNO_R3, Module:Arduino_UNO_R3, F.Cu at (147.3, 48.3)
- added A2: Adafruit_Feather_HUZZAH32_ESP32, Module:Adafruit_Feather, F.Cu at (143.5, 83.7)
- added C1: 470n, Capacitor_SMD:C_0603_1608Metric, F.Cu at (126.6, 33.1)
- added C2: 470n, Capacitor_SMD:C_0603_1608Metric, F.Cu at (138.7, 38.6)
- added C3: NOSTUFF, Capacitor_SMD:C_0603_1608Metric, F.Cu at (126.6, 31.3)
- added C4: NOSTUFF, Capacitor_SMD:C_0603_1608Metric, F.Cu at (138.7, 34.4)
- added C5: 10u, Capacitor_SMD:C_1206_3216Metric, F.Cu at (98.1, 63.5)
- added C6: 100n, Capacitor_SMD:C_0603_1608Metric, F.Cu at (100.7, 62.7)
- added C7: 10u, Capacitor_SMD:C_1206_3216Metric, F.Cu at (98.1, 68.6)
- added C8: 100n, Capacitor_SMD:C_0603_1608Metric, F.Cu at (100.7, 68.6)
- added J4: Conn_01x03, TerminalBlock_Phoenix:TerminalBlock_Phoenix_PT-1,5-3-3.5-H_1x03_P3.50mm_Horizontal, F.Cu at (131.1, 22.9)
- added J5: Conn_01x03, TerminalBlock_Phoenix:TerminalBlock_Phoenix_PT-1,5-3-3.5-H_1x03_P3.50mm_Horizontal, F.Cu at (143.2, 22.9)
- added L1: 600R/200mA, Inductor_SMD:L_0603_1608Metric, F.Cu at (125.9, 28.6)
- added L2: 600R/200mA, Inductor_SMD:L_0603_1608Metric, F.Cu at (138.7, 29.4)
- added R7: 200k, Resistor_SMD:R_0603_1608Metric, F.Cu at (127.0, 35.6)
- added R8: 200k, Resistor_SMD:R_0603_1608Metric, F.Cu at (133.8, 35.6)
- added U1: LM7805_TO220, Package_TO_SOT_THT:TO-220-3_Horizontal_TabDown, B.Cu at (103.2, 63.5)
- moved J2 79.6 mm to (124.5, 70.2), turned to -90 degrees
- moved J1 76.7 mm to (124.5, 84.1), turned to -90 degrees
- moved D2 68.5 mm to (132.3, 71.1), turned to -90 degrees
- moved D1 66.8 mm to (132.3, 76.2), turned to 90 degrees
- moved Q4 62.9 mm to (137.2, 69.3), turned to 180 degrees
- moved Q2 59.6 mm to (137.2, 78.0), turned to 180 degrees
- moved R6 58.0 mm to (140.5, 70.4), turned to 180 degrees
- moved R3 54.8 mm to (140.5, 79.0), turned to 180 degrees
- moved R5 49.1 mm to (147.3, 70.4), turned to 0 degrees
- moved R2 45.2 mm to (147.3, 79.0), turned to 0 degrees
- moved Q3 44.6 mm to (150.9, 70.4), turned to 180 degrees
- moved Q1 40.3 mm to (150.9, 79.0), turned to 180 degrees
- moved R4 39.7 mm to (154.2, 71.4), turned to 0 degrees
- moved R1 35.4 mm to (154.2, 80.0), turned to 0 degrees
- moved J3 30.2 mm to (159.0, 77.0), turned to 180 degrees
Routing:
- net GND: track 3.70 -> 15.2 mm
- net +12V: track 36.1 -> 41.8 mm
- net +5V: track 0.00 -> 5.69 mm
Other:
- board size 28.4 x 41.4 mm -> 68.6 x 53.3 mm
- net class Default removed

Commit message: WIP. Add relay LEDs, ui/display connection.
Parts:
- added D3: LED, LED_SMD:LED_0603_1608Metric, F.Cu at (163.8, 106.5)
- added D4: LED, LED_SMD:LED_0603_1608Metric, F.Cu at (148.2, 106.5)
- added J6: Conn_01x06_Female, Connector_PinHeader_2.54mm:PinHeader_1x06_P2.54mm_Vertical, F.Cu at (79.0, 60.5)
- added R10: 1k, Resistor_SMD:R_0603_1608Metric, F.Cu at (149.9, 106.5)
- added R9: 1k, Resistor_SMD:R_0603_1608Metric, F.Cu at (162.0, 106.5)
- moved J5 118.3 mm to (64.6, 111.2), turned to 0 degrees
- moved J4 103.7 mm to (76.8, 111.2), turned to 0 degrees
- moved L2 101.6 mm to (68.3, 102.6), turned to 90 degrees
- moved C4 96.9 mm to (67.6, 100.1), turned to 180 degrees
- moved C2 93.0 mm to (67.5, 98.4), turned to 180 degrees
- moved C5 90.7 mm to (145.8, 140.6), turned to 0 degrees
- moved R8 90.1 mm to (67.5, 96.6)
- moved C7 89.3 mm to (150.9, 140.6), turned to 180 degrees
- moved C6 87.4 mm to (145.0, 138.1), turned to 0 degrees
- moved L1 86.9 mm to (80.3, 102.6), turned to 90 degrees
- moved C8 85.7 mm to (150.9, 138.1), turned to 180 degrees
- moved U1 83.7 mm to (145.8, 135.5), turned to 0 degrees
- moved C3 83.4 mm to (79.6, 100.1), turned to 180 degrees
- moved C1 80.5 mm to (79.6, 98.4), turned to 180 degrees
- moved R7 77.3 mm to (79.6, 96.6), turned to 0 degrees
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Routing:
- net GND: track 15.2 -> 17.2 mm, vias 3 -> 5
- net /RELAY_UP+: track 12.0 -> 13.8 mm
- net /RELAY_DN+: track 12.0 -> 13.8 mm
- net Net-(D3-Pad2): track 0.00 -> 1.77 mm
- net Net-(D4-Pad2): track 0.00 -> 1.72 mm
Other:
- board size 68.6 x 53.3 mm -> 53.3 x 68.6 mm
- board text added: "DN"
- board text added: "Front UI LEDs"
- board text added: "UP"

Commit message: Add output enable, MCU wants relay up/down green LEDs.
Parts:
- added JP1: Jumper_2_Open, Connector_PinHeader_2.54mm:PinHeader_1x02_P2.54mm_Vertical, F.Cu at (157.2, 77.3)
- added JP2: Jumper_2_Bridged, Jumper:SolderJumper-2_P1.3mm_Bridged_RoundedPad1.0x1.5mm, B.Cu at (84.0, 73.2)
- added JP3: Jumper_2_Bridged, Jumper:SolderJumper-2_P1.3mm_Bridged_RoundedPad1.0x1.5mm, B.Cu at (74.0, 102.8)
- added LED3: LED_GRN, LED_SMD:LED_0603_1608Metric, F.Cu at (163.2, 66.8)
- added LED4: LED_GRN, LED_SMD:LED_0603_1608Metric, F.Cu at (149.2, 66.5)
- added Q5: MMBT3904L, Package_TO_SOT_SMD:SOT-23, F.Cu at (152.0, 71.0)
- added Q6: MMBT3904L, Package_TO_SOT_SMD:SOT-23, F.Cu at (160.8, 71.0)
- added R11: 10k, Resistor_SMD:R_0603_1608Metric, F.Cu at (153.0, 74.5)
- added R12: 10k, Resistor_SMD:R_0603_1608Metric, F.Cu at (161.8, 74.5)
- added R13: 1k, Resistor_SMD:R_0603_1608Metric, F.Cu at (163.2, 63.8)
- added R14: 1k, Resistor_SMD:R_0603_1608Metric, F.Cu at (151.2, 63.8)
- moved R1 20.8 mm to (161.6, 63.8)
- moved R4 20.8 mm to (153.0, 63.8)
- moved J3 20.8 mm to (158.5, 59.0)
- moved Q1 20.8 mm to (160.6, 67.1)
- moved Q3 20.8 mm to (151.9, 67.1)
- renumbered D3 to LED1, D4 to LED2
Connections:
- J4 pad 3: +5V -> /SENS_PWR
- J5 pad 3: +5V -> /SENS_PWR
- J6 pad 6: +5V -> /UI_PWR
- R2 pad 2: Net-(Q1-Pad3) -> Net-(R2-Pad2)
- R5 pad 2: Net-(Q3-Pad3) -> Net-(R5-Pad2)
Routing:
- net Net-(R2-Pad2): track 0.00 -> 19.7 mm
- net Net-(R5-Pad2): track 0.00 -> 19.4 mm
- net /EN_OUTPUT: track 0.00 -> 9.24 mm, vias 0 -> 1
- net Net-(Q6-Pad1): track 0.00 -> 3.63 mm
- net Net-(Q5-Pad1): track 0.00 -> 3.63 mm
- net Net-(LED4-Pad2): track 0.00 -> 2.47 mm
- net GND: track 17.2 -> 19.6 mm, vias 5 -> 6
- net /EN_RELAY_DN: track 5.20 -> 6.91 mm
- net /EN_RELAY_UP: track 5.20 -> 6.87 mm
- net Net-(LED3-Pad2): track 0.00 -> 1.39 mm
- net Net-(Q3-Pad3): track 1.73 -> 2.36 mm
- net Net-(Q1-Pad3): track 1.73 -> 2.32 mm

Commit message: Line up inverter, output enable transistors.
Parts:
- moved LED3 5.59 mm to (160.8, 61.8), turned to 0 degrees
- moved LED4 5.49 mm to (152.0, 61.8), turned to 180 degrees
- moved R13 2.55 mm to (160.8, 63.2), turned to 180 degrees
- moved R4 1.37 mm to (152.0, 64.8), turned to 0 degrees
- moved R1 1.29 mm to (160.8, 64.8), turned to 180 degrees
- moved R14 0.90 mm to (152.0, 63.2), turned to 0 degrees
- moved Q5 0.25 mm to (152.0, 70.8), turned to 180 degrees
- moved Q6 0.25 mm to (160.8, 70.8), turned to 180 degrees
- moved Q1 0.22 mm to (160.8, 67.2), turned to 0 degrees
- moved Q3 0.14 mm to (152.0, 67.2), turned to 0 degrees
Routing:
- net Net-(Q6-Pad1): track 3.63 -> 2.00 mm
- net Net-(Q5-Pad1): track 3.63 -> 2.00 mm
- net Net-(R5-Pad2): track 19.4 -> 20.8 mm
- net Net-(Q1-Pad1): track 1.57 -> 2.80 mm
- net Net-(LED4-Pad2): track 2.47 -> 1.52 mm
- net Net-(R2-Pad2): track 19.7 -> 20.5 mm
- net /EN_RELAY_DN: track 6.91 -> 7.46 mm
- net GND: track 19.6 -> 19.3 mm, vias 6 -> 7

Commit message: Swap CLK and LE pins on LED UI display connection.
Parts:
- moved J6 1.51 mm to (80.5, 60.6)
Connections:
- net /UI_PWR renamed /UI_VDD
- J6 pad 3: /LE -> /CLK
- J6 pad 4: /CLK -> /LE

Commit message: Add Up/Down buttons switch input with hardware debounce.
HW debounce copied from ultrasonic PCB project.
Parts:
- added C10: 1uF, Capacitor_SMD:C_0603_1608Metric, F.Cu at (46.3, 54.2)
- added C11: 1uF, Capacitor_SMD:C_0603_1608Metric, F.Cu at (42.7, 54.2)
- added C12: 1uF, Capacitor_SMD:C_0603_1608Metric, F.Cu at (42.7, 56.0)
- added C9: 1uF, Capacitor_SMD:C_0603_1608Metric, F.Cu at (46.3, 56.0)
- added D3: LL4148, Diode_SMD:D_MiniMELF, F.Cu at (48.8, 52.2)
- added D4: LL4148, Diode_SMD:D_MiniMELF, F.Cu at (40.2, 52.2)
- added J7: Conn_01x04_Female, TerminalBlock_Phoenix:TerminalBlock_Phoenix_PT-1,5-4-3.5-H_1x04_P3.50mm_Horizontal, F.Cu at (49.8, 45.0)
- added JP3: Jumper_2_Bridged, Jumper:SolderJumper-2_P1.3mm_Bridged_RoundedPad1.0x1.5mm, F.Cu at (52.5, 60.0)
- added R15: 6.8k, Resistor_SMD:R_0603_1608Metric, F.Cu at (52.2, 54.2)
- added R16: 8.2k, Resistor_SMD:R_0603_1608Metric, F.Cu at (49.2, 54.2)
- added R17: 6.8k, Resistor_SMD:R_0603_1608Metric, F.Cu at (36.7, 54.2)
- added R18: 8.2k, Resistor_SMD:R_0603_1608Metric, F.Cu at (39.7, 54.2)
- added R19: 4k7, Resistor_SMD:R_0603_1608Metric, F.Cu at (45.2, 63.7)
- added R20: 4k7, Resistor_SMD:R_0603_1608Metric, F.Cu at (43.8, 63.7)
- added U2: NC7WZ14P6X, Package_TO_SOT_SMD:SOT-363_SC-70-6, F.Cu at (44.5, 60.0)
- J6: footprint Connector_PinHeader_2.54mm:PinHeader_1x06_P2.54mm_Vertical -> TerminalBlock_Phoenix:TerminalBlock_Phoenix_PT-1,5-6-3.5-H_1x06_P3.50mm_Horizontal
- moved J6 23.3 mm to (97.8, 45.0), turned to 180 degrees
- moved JP2 16.0 mm to (84.0, 57.3)
- renumbered JP3 to JP4
Connections:
- net /UI_VDD renamed /UI_PWR
- A1 pad 17: unconnected-(A1-Pad17) -> /BTN_DN
- A1 pad 18: unconnected-(A1-Pad18) -> /BTN_UP
Other:
- board text added: "Angle Sensors"
- board text added: "Up/Down Buttons"

Commit message: Fix hardware debounce circuit (was incorrect).
Connections:
- U2 pad 1: /HWDebounce/SW1IN -> Net-(C10-Pad1)
- U2 pad 3: /HWDebounce/SW2IN -> Net-(C11-Pad1)
Changed lines of the file:
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@@
     (fp_line (start 0.675 -1.1) (end -0.175 -1.1) (layer "F.Fab") (width 0.1))
     (pad "1" smd rect locked (at -0.95 -0.65 270) (size 0.65 0.4) (layers "F.Cu" "F.Paste" "F.Mask")
-      (net 85 "/HWDebounce/SW1IN") (pinfunction "A1") (pintype "input"))
+      (net 70 "Net-(C10-Pad1)") (pinfunction "A1") (pintype "input"))
     (pad "2" smd rect locked (at -0.95 0 270) (size 0.65 0.4) (layers "F.Cu" "F.Paste" "F.Mask")
       (net 1 "GND") (pinfunction "GND") (pintype "passive"))
     (pad "3" smd rect locked (at -0.95 0.65 270) (size 0.65 0.4) (layers "F.Cu" "F.Paste" "F.Mask")
-      (net 86 "/HWDebounce/SW2IN") (pinfunction "A2") (pintype "input"))
+      (net 84 "Net-(C11-Pad1)") (pinfunction "A2") (pintype "input"))
     (pad "4" smd rect locked (at 0.95 0.65 270) (size 0.65 0.4) (layers "F.Cu" "F.Paste" "F.Mask")
       (net 90 "Net-(R20-Pad2)") (pinfunction "Y2") (pintype "output"))

Commit message: Flip Arduino UNO R3 footprint.
Parts:
- A1: moved to B.Cu
- moved A1 48.5 mm to (179.1, 91.4)
