File: power-wedge-control.kicad_pcb (KiCad board)
At the start: 2 copper layers, 77.2 x 64.5 mm, 71 parts, among them J1 Conn_01x02, J2 Conn_01x03, J3 Conn_01x02, J4 Conn_01x03, J5 Conn_01x03, J6 Conn_01x06_Female, J7 Conn_01x04_Female, J8 Conn_01x03, J9 MicroSD_Hirose_DM3D-SF, Q1 MMBT3904L, Q2 DMP3099L, Q3 MMBT3904L, Q4 DMP3099L, Q5 MMBT3904L, Q6 MMBT3904L, U1 LM7805_TO220, U2 NC7WZ14P6X, U3 TLV70233DBV, U5 NC7WZ17P6X, U6 NC7WZ17P6X

Commit message: Change 5V regulator LM7805 to LM1117.
Parts:
- U1: value LM7805_TO220 -> LM1117-5.0; footprint Package_TO_SOT_THT:TO-220-3_Horizontal_TabDown -> Package_TO_SOT_SMD:TO-252-2
- moved C7 17.8 mm to (141.9, 98.9)
- moved C8 17.7 mm to (141.1, 96.9)
- moved C5 13.2 mm to (137.0, 103.6), turned to 90 degrees
- moved U1 13.0 mm to (143.8, 103.6)
- moved C6 12.0 mm to (139.2, 103.6), turned to 90 degrees
- moved U3 11.2 mm to (139.5, 94.3), turned to 180 degrees
- moved C15 10.3 mm to (138.0, 96.9), turned to 0 degrees
- moved C14 10.3 mm to (137.2, 98.9), turned to 0 degrees
Connections:
- U1 pad 1: +12V -> GND
- U1 pad 2: GND -> +5V
- U1 pad 3: +5V -> +12V
Routing:
- net GND: track 54.7 -> 73.0 mm, vias 26 -> 30
- net +5V: track 56.1 -> 38.0 mm
- net +12V: track 87.4 -> 101.0 mm
- net +3V3: track 47.1 -> 38.2 mm
Other:
- board text added: "3.3V"

Commit message: Flip J3 relay test points away from Uno USB connector.
Parts:
- moved J3 3.71 mm to (120.0, 100.7), turned to -90 degrees
Connections:
- J3 pad 1: /EN_RELAY_UP -> /EN_RELAY_DN
- J3 pad 2: /EN_RELAY_DN -> /EN_RELAY_UP
Routing:
- net /EN_RELAY_UP: track 10.3 -> 7.06 mm
- net /EN_RELAY_DN: track 8.64 -> 7.09 mm
Changed lines of the file:
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@@
       (effects (font (size 0.4 0.4) (thickness 0.06)))
     )
+    (fp_line (start 0 -1.56) (end 0.8 -1.56) (layer "F.SilkS") (width 0.12))
     (fp_line (start 0 1.56) (end -0.8 1.56) (layer "F.SilkS") (width 0.12))
+    (fp_line (start 0 -1.56) (end -1.8 -1.56) (layer "F.SilkS") (width 0.12))
     (fp_line (start 0 1.56) (end 0.8 1.56) (layer "F.SilkS") (width 0.12))
-    (fp_line (start 0 -1.56) (end 0.8 -1.56) (layer "F.SilkS") (width 0.12))
-    (fp_line (start 0 -1.56) (end -1.8 -1.56) (layer "F.SilkS") (width 0.12))
+    (fp_line (start 2.05 -1.7) (end -2.05 -1.7) (layer "F.CrtYd") (width 0.05))
+    (fp_line (start 2.05 1.7) (end 2.05 -1.7) (layer "F.CrtYd") (width 0.05))
     (fp_line (start -2.05 1.7) (end 2.05 1.7) (layer "F.CrtYd") (width 0.05))
     (fp_line (start -2.05 -1.7) (end -2.05 1.7) (layer "F.CrtYd") (width 0.05))
-    (fp_line (start 2.05 -1.7) (end -2.05 -1.7) (layer "F.CrtYd") (width 0.05))
-    (fp_line (start 2.05 1.7) (end 2.05 -1.7) (layer "F.CrtYd") (width 0.05))
+    (fp_line (start 0.8 -1.45) (end 0.8 1.45) (layer "F.Fab") (width 0.1))
     (fp_line (start 0.8 1.45) (end -0.8 1.45) (layer "F.Fab") (width 0.1))
-    (fp_line (start 0.8 -1.45) (end 0.8 1.45) (layer "F.Fab") (width 0.1))
     (fp_line (start -0.8 1.45) (end -0.8 -1.05) (layer "F.Fab") (width 0.1))
+    (fp_line (start -0.8 -1.05) (end -0.4 -1.45) (layer "F.Fab") (width 0.1))
     (fp_line (start -0.4 -1.45) (end 0.8 -1.45) (layer "F.Fab") (width 0.1))
-    (fp_line (start -0.8 -1.05) (end -0.4 -1.45) (layer "F.Fab") (width 0.1))
     (pad "1" smd roundrect locked (at -1.1375 -0.95 180) (size 1.325 0.6) (layers "F.Cu" "F.Paste" "F.Mask") (roundrect_rratio 0.25)
       (net 16 "+5V") (pinfunction "IN") (pintype "input"))
@@
   )
   (footprint "Connector_PinHeader_2.54mm:PinHeader_1x02_P2.54mm_Horizontal" (layer "B.Cu")
-    (at 122.5935 103.3556 90)
+    (at 120 100.7 -90)
     (descr "Through hole angled pin header, 1x02, 2.54mm pitch, 6mm pin length, single row")
     (tags "Through hole angled pin header THT 1x02 2.54mm single row")
@@
     (fp_line (start 4.04 1.27) (end 4.04 -3.81) (layer "B.Fab") (width 0.1))
     (fp_line (start -0.32 0.32) (end -0.32 -0.32) (layer "B.Fab") (width 0.1))
-    (pad "1" thru_hole rect locked (at 0 0 90) (size 1.7 1.7) (drill 1) (layers *.Cu *.Mask)
-      (net 5 "/EN_RELAY_UP") (pinfunction "Pin_1") (pintype "passive"))
-    (pad "2" thru_hole oval locked (at 0 -2.54 90) (size 1.7 1.7) (drill 1) (layers *.Cu *.Mask)
-      (net 6 "/EN_RELAY_DN") (pinfunction "Pin_2") (pintype "passive"))
+    (pad "1" thru_hole rect locked (at 0 0 270) (size 1.7 1.7) (drill 1) (layers *.Cu *.Mask)
+      (net 6 "/EN_RELAY_DN") (pinfunction "Pin_1") (pintype "passive"))
+    (pad "2" thru_hole oval locked (at 0 -2.54 270) (size 1.7 1.7) (drill 1) (layers *.Cu *.Mask)
+      (net 5 "/EN_RELAY_UP") (pinfunction "Pin_2") (pintype "passive"))
     (model "${KICAD6_3DMODEL_DIR}/Connector_PinHeader_2.54mm.3dshapes/PinHeader_1x02_P2.54mm_Horizontal.wrl"
       (offset (xyz 0 0 0))
@@
     (effects (font (size 1.5 1.5) (thickness 0.3)) (justify right mirror))
   )
-  (gr_text "EN\nOUT" (at 118.872 109.728) (layer "B.SilkS")
+  (gr_text "EN\nOUT" (at 116.7 119.6) (layer "B.SilkS")
     (effects (font (size 1.5 1.5) (thickness 0.3)) (justify mirror))
   )
@@
   (segment (start 149.14782 124.5) (end 144.451623 124.5) (width 0.8) (layer "B.Cu") (net 4))
   (segment (start 144.451623 124.5) (end 144.450741 124.499118) (width 0.8) (layer "B.Cu") (net 4))
-  (segment (start 124.1329 104.895) (end 122.5935 103.3556) (width 0.3) (layer "F.Cu") (net 5))
-  (segment (start 122.5935 103.3556) (end 122.5935 97.406838) (width 0.3) (layer "F.Cu") (net 5))
   (segment (start 124.8347 104.895) (end 124.8347 106.395) (width 0.3) (layer "F.Cu") (net 5))
+  (segment (start 122.54 100.7) (end 122.54 103.3021) (width 0.3) (layer "F.Cu") (net 5))
   (segment (start 124.8347 104.895) (end 124.1329 104.895) (width 0.3) (layer "F.Cu") (net 5))
-  (segment (start 118.5141 104.895) (end 120.0535 103.3556) (width 0.3) (layer "F.Cu") (net 6))
+  (segment (start 122.54 103.3021) (end 124.1329 104.895) (width 0.3) (layer "F.Cu") (net 5))
+  (segment (start 120 103.4091) (end 118.5141 104.895) (width 0.3) (layer "F.Cu") (net 6))
   (segment (start 117.7347 104.895) (end 117.7347 106.395) (width 0.3) (layer "F.Cu") (net 6))
-  (segment (start 120.0535 103.3556) (end 120.0535 99.1697) (width 0.3) (layer "F.Cu") (net 6))
   (segment (start 117.7347 104.895) (end 118.5141 104.895) (width 0.3) (layer "F.Cu") (net 6))
+  (segment (start 120 100.7) (end 120 103.4091) (width 0.3) (layer "F.Cu") (net 6))
   (segment (start 126.5972 108.895) (end 126.5972 111.445) (width 0.3) (layer "F.Cu") (net 7))
   (segment (start 126.4847 107.07) (end 125.6097 107.945) (width 0.3) (layer "F.Cu") (net 8))

Commit message: Change 7SegDisp UI connection pin labels for TLC6C5912.
Connections:
- net /CLK renamed /RCK
- net /LE renamed /G
- net /OE renamed /SER_IN
- net /SDI renamed /SRCK
Other:
- board text added: "G"
- board text added: "RCK"
- board text added: "SER"
- board text added: "SRK"
- board text removed: "CLK"
- board text removed: "LE"
- board text removed: "OE"
- board text removed: "SDI"
Changed lines of the file:
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@@
   (net 63 "/EN_OUTPUT")
   (net 64 "Net-(C10-Pad1)")
-  (net 65 "/SDI")
-  (net 66 "/LE")
-  (net 67 "/CLK")
-  (net 68 "/OE")
+  (net 65 "/SER_IN")
+  (net 66 "/G")
+  (net 67 "/RCK")
+  (net 68 "/SRCK")
   (net 69 "Net-(LED1-Pad2)")
   (net 70 "Net-(Q5-Pad1)")
@@
       (effects (font (size 0.4 0.4) (thickness 0.06)))
     )
-    (fp_line (start 0 -1.56) (end 0.8 -1.56) (layer "F.SilkS") (width 0.12))
-    (fp_line (start 0 1.56) (end -0.8 1.56) (layer "F.SilkS") (width 0.12))
     (fp_line (start 0 -1.56) (end -1.8 -1.56) (layer "F.SilkS") (width 0.12))
     (fp_line (start 0 1.56) (end 0.8 1.56) (layer "F.SilkS") (width 0.12))
-    (fp_line (start 2.05 -1.7) (end -2.05 -1.7) (layer "F.CrtYd") (width 0.05))
+    (fp_line (start 0 -1.56) (end 0.8 -1.56) (layer "F.SilkS") (width 0.12))
+    (fp_line (start 0 1.56) (end -0.8 1.56) (layer "F.SilkS") (width 0.12))
     (fp_line (start 2.05 1.7) (end 2.05 -1.7) (layer "F.CrtYd") (width 0.05))
-    (fp_line (start -2.05 1.7) (end 2.05 1.7) (layer "F.CrtYd") (width 0.05))
     (fp_line (start -2.05 -1.7) (end -2.05 1.7) (layer "F.CrtYd") (width 0.05))
-    (fp_line (start 0.8 -1.45) (end 0.8 1.45) (layer "F.Fab") (width 0.1))
-    (fp_line (start 0.8 1.45) (end -0.8 1.45) (layer "F.Fab") (width 0.1))
+    (fp_line (start -2.05 1.7) (end 2.05 1.7) (layer "F.CrtYd") (width 0.05))
+    (fp_line (start 2.05 -1.7) (end -2.05 -1.7) (layer "F.CrtYd") (width 0.05))
     (fp_line (start -0.8 1.45) (end -0.8 -1.05) (layer "F.Fab") (width 0.1))
     (fp_line (start -0.8 -1.05) (end -0.4 -1.45) (layer "F.Fab") (width 0.1))
+    (fp_line (start 0.8 -1.45) (end 0.8 1.45) (layer "F.Fab") (width 0.1))
+    (fp_line (start 0.8 1.45) (end -0.8 1.45) (layer "F.Fab") (width 0.1))
     (fp_line (start -0.4 -1.45) (end 0.8 -1.45) (layer "F.Fab") (width 0.1))
     (pad "1" smd roundrect locked (at -1.1375 -0.95 180) (size 1.325 0.6) (layers "F.Cu" "F.Paste" "F.Mask") (roundrect_rratio 0.25)
@@
       (net 1 "GND") (pinfunction "Pin_1") (pintype "passive"))
     (pad "2" thru_hole circle locked (at 3.5 0) (size 2.4 2.4) (drill 1.2) (layers *.Cu *.Mask)
-      (net 65 "/SDI") (pinfunction "Pin_2") (pintype "passive"))
+      (net 68 "/SRCK") (pinfunction "Pin_2") (pintype "passive"))
     (pad "3" thru_hole circle locked (at 7 0) (size 2.4 2.4) (drill 1.2) (layers *.Cu *.Mask)
-      (net 67 "/CLK") (pinfunction "Pin_3") (pintype "passive"))
+      (net 67 "/RCK") (pinfunction "Pin_3") (pintype "passive"))
     (pad "4" thru_hole circle locked (at 10.5 0) (size 2.4 2.4) (drill 1.2) (layers *.Cu *.Mask)
-      (net 66 "/LE") (pinfunction "Pin_4") (pintype "passive"))
+      (net 66 "/G") (pinfunction "Pin_4") (pintype "passive"))
     (pad "5" thru_hole circle locked (at 14 0) (size 2.4 2.4) (drill 1.2) (layers *.Cu *.Mask)
-      (net 68 "/OE") (pinfunction "Pin_5") (pintype "passive"))
+      (net 65 "/SER_IN") (pinfunction "Pin_5") (pintype "passive"))
     (pad "6" thru_hole circle locked (at 17.5 0) (size 2.4 2.4) (drill 1.2) (layers *.Cu *.Mask)
       (net 81 "/UI_PWR") (pinfunction "Pin_6") (pintype "passive"))
@@
       (net 6 "/EN_RELAY_DN") (pinfunction "D3") (pintype "bidirectional"))
     (pad "19" thru_hole oval locked (at 25.4 -48.26 270) (size 1.6 1.6) (drill 1) (layers *.Cu *.Mask)
-      (net 68 "/OE") (pinfunction "D4") (pintype "bidirectional"))
+      (net 65 "/SER_IN") (pinfunction "D4") (pintype "bidirectional"))
     (pad "20" thru_hole oval locked (at 22.86 -48.26 270) (size 1.6 1.6) (drill 1) (layers *.Cu *.Mask)
-      (net 66 "/LE") (pinfunction "D5") (pintype "bidirectional"))
+      (net 66 "/G") (pinfunction "D5") (pintype "bidirectional"))
     (pad "21" thru_hole oval locked (at 20.32 -48.26 270) (size 1.6 1.6) (drill 1) (layers *.Cu *.Mask)
-      (net 67 "/CLK") (pinfunction "D6") (pintype "bidirectional"))
+      (net 67 "/RCK") (pinfunction "D6") (pintype "bidirectional"))
     (pad "22" thru_hole oval locked (at 17.78 -48.26 270) (size 1.6 1.6) (drill 1) (layers *.Cu *.Mask)
-      (net 65 "/SDI") (pinfunction "D7") (pintype "bidirectional"))
+      (net 68 "/SRCK") (pinfunction "D7") (pintype "bidirectional"))
     (pad "23" thru_hole oval locked (at 13.72 -48.26 270) (size 1.6 1.6) (drill 1) (layers *.Cu *.Mask)
       (net 19 "/BTN_DN") (pinfunction "D8") (pintype "bidirectional"))
@@
   (gr_line (start 113.538 141.045) (end 113.538 76.581) (layer "Edge.Cuts") (width 0.05))
   (gr_line (start 113.538 76.581) (end 190.754 76.581) (layer "Edge.Cuts") (width 0.05))
-  (gr_text "CLK" (at 141.5288 136.2456 270) (layer "B.SilkS")
+  (gr_text "RCK" (at 141.5288 136.2456 270) (layer "B.SilkS")
     (effects (font (size 1.5 1.5) (thickness 0.3)) (justify right mirror))
   )
@@
     (effects (font (size 1.5 1.5) (thickness 0.3)) (justify mirror))
   )
-  (gr_text "OE" (at 148.5392 136.2456 270) (layer "B.SilkS")
+  (gr_text "SER" (at 148.5392 136.2456 270) (layer "B.SilkS")
     (effects (font (size 1.5 1.5) (thickness 0.3)) (justify right mirror))
   )
@@
     (effects (font (size 1.5 1.5) (thickness 0.3)) (justify mirror))
   )
-  (gr_text "SDI" (at 138.0744 136.1948 270) (layer "B.SilkS")
+  (gr_text "SRK" (at 138.0744 136.1948 270) (layer "B.SilkS")
     (effects (font (size 1.5 1.5) (thickness 0.3)) (justify right mirror))
   )
@@
     (effects (font (size 1.5 1.5) (thickness 0.3)) (justify mirror))
   )
-  (gr_text "LE" (at 145.034 136.2964 270) (layer "B.SilkS")
+  (gr_text "G" (at 145.034 136.2964 270) (layer "B.SilkS")
     (effects (font (size 1.5 1.5) (thickness 0.3)) (justify right mirror))
   )
@@
   (segment (start 160.329 116.778) (end 160.329 120.4) (width 0.3) (layer "F.Cu") (net 64))
   (segment (start 161.146 115.254) (end 160.329 116.071) (width 0.3) (layer "F.Cu") (net 64))
-  (segment (start 145.65024 129.726822) (end 145.650241 124.099998) (width 0.3) (layer "F.Cu") (net 65))
-  (segment (start 145.650241 124.099998) (end 145.650243 117.018343) (width 0.3) (layer "F.Cu") (net 65))
-  (segment (start 143.977062 131.4) (end 145.65024 129.726822) (width 0.3) (layer "F.Cu") (net 65))
-  (segment (start 145.650243 117.018343) (end 167.767 94.901586) (width 0.3) (layer "F.Cu") (net 65))
-  (segment (start 137.9988 134.6554) (end 141.2542 131.4) (width 0.3) (layer "F.Cu") (net 65))
-  (segment (start 167.767 94.901586) (end 167.767 79.375) (width 0.3) (layer "F.Cu") (net 65))
-  (segment (start 141.2542 131.4) (end 143.977062 131.4) (width 0.3) (layer "F.Cu") (net 65))
+  (segment (start 175.387 89.613) (end 175.387 79.375) (width 0.3) (layer "F.Cu") (net 65))
+  (segment (start 148.4988 134.6554) (end 147.2988 133.4554) (width 0.3) (layer "F.Cu") (net 65))
+  (segment (start 147.2988 133.4554) (end 147.2988 117.7012) (width 0.3) (layer "F.Cu") (net 65))
+  (segment (start 147.2988 117.7012) (end 175.387 89.613) (width 0.3) (layer "F.Cu") (net 65))
   (segment (start 146.749281 117.473581) (end 172.847 91.375862) (width 0.3) (layer "F.Cu") (net 66))
   (segment (start 144.9988 134.6554) (end 146.74928 132.90492) (width 0.3) (layer "F.Cu") (net 66))
@@
   (segment (start 146.19976 129.95444) (end 146.19976 127.8) (width 0.3) (layer "F.Cu") (net 67))
   (segment (start 146.19976 127.8) (end 146.199762 117.245962) (width 0.3) (layer "F.Cu") (net 67))
-  (segment (start 175.387 89.613) (end 175.387 79.375) (width 0.3) (layer "F.Cu") (net 68))
-  (segment (start 148.4988 134.6554) (end 147.2988 133.4554) (width 0.3) (layer "F.Cu") (net 68))
-  (segment (start 147.2988 133.4554) (end 147.2988 117.7012) (width 0.3) (layer "F.Cu") (net 68))
-  (segment (start 147.2988 117.7012) (end 175.387 89.613) (width 0.3) (layer "F.Cu") (net 68))
+  (segment (start 145.65024 129.726822) (end 145.650241 124.099998) (width 0.3) (layer "F.Cu") (net 68))
+  (segment (start 145.650241 124.099998) (end 145.650243 117.018343) (width 0.3) (layer "F.Cu") (net 68))
+  (segment (start 143.977062 131.4) (end 145.65024 129.726822) (width 0.3) (layer "F.Cu") (net 68))
+  (segment (start 145.650243 117.018343) (end 167.767 94.901586) (width 0.3) (layer "F.Cu") (net 68))
+  (segment (start 137.9988 134.6554) (end 141.2542 131.4) (width 0.3) (layer "F.Cu") (net 68))
+  (segment (start 167.767 94.901586) (end 167.767 79.375) (width 0.3) (layer "F.Cu") (net 68))
+  (segment (start 141.2542 131.4) (end 143.977062 131.4) (width 0.3) (layer "F.Cu") (net 68))
   (segment (start 121.5095 126.7968) (end 123.0843 128.3716) (width 0.3) (layer "F.Cu") (net 69))
   (segment (start 121.4718 126.7968) (end 121.5095 126.7968) (width 0.3) (layer "F.Cu") (net 69))

Commit message: Move power supply near angle sensors. Swap several MCU pins.
Move button debounce up near MCU pins.
Add top layer zones for thermal at voltage regs.
Parts:
- JP4: moved to F.Cu
- moved JP3 31.4 mm to (182.9, 92.1), turned to 90 degrees
- moved C10 27.6 mm to (172.2, 93.1)
- moved C11 27.6 mm to (175.7, 93.1)
- moved C12 27.6 mm to (175.8, 91.4)
- moved C9 27.6 mm to (172.2, 91.4)
- moved D3 27.6 mm to (169.7, 95.1)
- moved D4 27.6 mm to (178.2, 95.1)
- moved R15 27.6 mm to (169.0, 91.4)
- moved R16 27.6 mm to (169.0, 93.1)
- moved R17 27.6 mm to (178.9, 91.4)
- moved R18 27.6 mm to (178.9, 93.1)
- moved R19 27.6 mm to (173.2, 85.6)
- moved R20 27.6 mm to (174.7, 85.6)
- moved U2 27.6 mm to (173.9, 89.0)
- moved C14 19.7 mm to (153.7, 109.7)
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Connections:
- A1 pad 17: /EN_RELAY_UP -> /EN_RELAY_DN
- A1 pad 18: /EN_RELAY_DN -> /EN_RELAY_UP
- A1 pad 19: /SER_IN -> /BTN_DN
- A1 pad 20: /G -> /BTN_UP
- A1 pad 21: /RCK -> /SER_IN
- A1 pad 22: /SRCK -> /G
- A1 pad 23: /BTN_DN -> /RCK
- A1 pad 24: /BTN_UP -> /SRCK
- JP2 pad 1: +5V -> +3V3
Routing:
- net +5V: track 38.0 -> 115.9 mm
- net /EN_RELAY_DN: track 7.09 -> 83.4 mm, vias 0 -> 2
- net /HWDebounce/SW2IN: track 19.5 -> 92.7 mm
- net /EN_RELAY_UP: track 7.06 -> 78.3 mm, vias 0 -> 2
- net GND: track 73.0 -> 118.3 mm, vias 30 -> 47
- net +3V3: track 38.2 -> 72.9 mm, vias 4 -> 6
- net /HWDebounce/SW1IN: track 39.4 -> 72.2 mm
- net /BTN_DN: track 33.3 -> 5.68 mm, vias 2 -> 0
- net /BTN_UP: track 32.3 -> 5.55 mm, vias 2 -> 0
- net /SENS_PWR: track 53.1 -> 39.8 mm, vias 1 -> 0
- net +12V: track 101.0 -> 89.1 mm
- net /BTN_PWR: track 15.0 -> 20.7 mm
- net /UI_PWR: track 29.6 -> 24.5 mm
- net /SER_IN: track 67.4 -> 72.4 mm
- net /G: track 66.8 -> 70.7 mm
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- added copper zone on F.Cu, net +12V
- added copper zone on F.Cu, net +3V3
- added copper zone on F.Cu, net +5V
- added copper zone on F.Cu, net GND

Commit message: Add ferrite bead on sensor power.
Parts:
- removed JP4: Jumper_2_Bridged, Jumper:SolderJumper-2_P1.3mm_Bridged_RoundedPad1.0x1.5mm
- added L3: 600R/200mA, Inductor_SMD:L_0603_1608Metric, F.Cu at (174.2, 114.1)
Routing:
- net /SENS_PWR: track 39.8 -> 39.3 mm

Commit message: Add GND to angle sensor test points.
Parts:
- J8: value Conn_01x03 -> Conn_01x04; footprint Connector_PinHeader_2.54mm:PinHeader_1x03_P2.54mm_Horizontal -> Connector_PinHeader_2.54mm:PinHeader_1x04_P2.54mm_Horizontal
Other:
- board text added: "GND ANGL2 5V ANGL1"

Commit message: WIP. Add support for active-high (15V max) switch input to schematic.
Parts:
- added JP4: SW_SPDT, Jumper:SolderJumper-3_P2.0mm_Open_TrianglePad1.0x1.5mm, B.Cu at (136.3, 109.7)
- added JP5: SW_SPDT, Jumper:SolderJumper-3_P2.0mm_Open_TrianglePad1.0x1.5mm, B.Cu at (136.3, 104.1)
- added Q7: MMBT3904L, Package_TO_SOT_SMD:SOT-23, F.Cu at (139.3, 110.1)
- added Q8: MMBT3904L, Package_TO_SOT_SMD:SOT-23, F.Cu at (136.8, 103.5)
- added R21: 220k, Resistor_SMD:R_0603_1608Metric, F.Cu at (136.7, 112.6)
- added R22: 220k, Resistor_SMD:R_0603_1608Metric, F.Cu at (131.5, 105.5)
- added R23: 10k, Resistor_SMD:R_0603_1608Metric, F.Cu at (139.8, 112.6)
- added R24: 10k, Resistor_SMD:R_0603_1608Metric, F.Cu at (133.1, 105.5)
- added U4: 4050, Package_SO:SOIC-16W_5.3x10.2mm_P1.27mm, F.Cu at (135.8, 117.9)
Connections:
- D3 pad 2: /HWDebounce/SW1IN -> /~{SW1}
- D4 pad 2: /HWDebounce/SW2IN -> /~{SW2}
- J7 pad 1: /HWDebounce/SW1IN -> /SW1EXT
- J7 pad 4: /HWDebounce/SW2IN -> /SW2EXT
- R15 pad 1: /HWDebounce/SW1IN -> /~{SW1}
- R16 pad 2: /HWDebounce/SW1IN -> /~{SW1}
- R17 pad 1: /HWDebounce/SW2IN -> /~{SW2}
- R18 pad 2: /HWDebounce/SW2IN -> /~{SW2}
Routing:
- net /HWDebounce/SW2IN: track 92.7 -> 0.00 mm
- net /~{SW2}: track 0.00 -> 90.9 mm
- net /HWDebounce/SW1IN: track 72.2 -> 0.00 mm
- net /~{SW1}: track 0.00 -> 70.4 mm
- net +5V: track 115.7 -> 121.5 mm
Other:
- board text added: "15V Max Active-High"
- board text added: "Buttons Switch Mode"
- board text added: "Contact Closure"
- board text added: "Don't apply voltage to + unless in this mode."
- board text added: "Normal contact closure between + and GND."

Commit message: Add support for active-high (15V max) switch input to PCB layout.
Parts:
- moved JP3 18.7 mm to (164.9, 97.3)
- moved Q8 4.29 mm to (135.6, 107.6), turned to 90 degrees
- moved R24 3.91 mm to (133.1, 109.4)
- moved R22 1.80 mm to (133.1, 106.4), turned to -90 degrees
Routing:
- net /SW2EXT: track 0.00 -> 59.6 mm, vias 0 -> 3
- net /BTN_PWR: track 20.7 -> 68.0 mm, vias 1 -> 3
- net /SW1EXT: track 0.00 -> 42.0 mm, vias 0 -> 3
- net /~{SW2}: track 90.9 -> 60.0 mm, vias 0 -> 3
- net /~{SW1}: track 70.4 -> 48.1 mm, vias 0 -> 3
- net +5V: track 121.5 -> 99.3 mm
- net GND: track 118.3 -> 131.1 mm, vias 47 -> 56
- net /SW2IN_15V: track 0.00 -> 12.6 mm, vias 0 -> 1
- net /SW1IN_15V: track 0.00 -> 7.15 mm, vias 0 -> 1
- net Net-(R24-Pad2): track 0.00 -> 4.43 mm
- net Net-(R23-Pad2): track 0.00 -> 1.79 mm
- net Net-(Q7-Pad1): track 0.00 -> 1.68 mm
- net Net-(Q8-Pad1): track 0.00 -> 1.55 mm
- net /G: track 70.7 -> 72.1 mm
- net /SER_IN: track 72.4 -> 73.8 mm
