File: power-wedge-control.kicad_pcb (KiCad board)
At the start: 2 copper layers, 77.2 x 64.5 mm, 81 parts, among them J1 Conn_01x02, J10 Conn_01x10, J11 Conn_01x08, J12 Conn_01x06, J2 Conn_01x03, J3 Conn_01x02, J4 Conn_01x03, J5 Conn_01x03, J6 Conn_01x06_Female, J7 Conn_01x04_Female, J8 Conn_01x04, J9 MicroSD_Hirose_DM3D-SF, Q1 MMBT3904L, Q2 DMP3099L, Q3 MMBT3904L, Q4 DMP3099L, Q5 MMBT3904L, Q6 MMBT3904L, U1 LM1117-5.0, U2 NC7WZ14P6X, U3 TLV70233DBV, U4 LTV-817S, U5 NC7WZ17P6X, U6 NC7WZ17P6X, U7 LTV-817S

Commit message: Add hardware manual control option to schematic and WIP layout.
TODO: 4-wires to up/down buttons: +12V, GND, UP input, DN input.
TODO: EN manual to MCU input pin.
TODO: EN manual test/engr pin.
Parts:
- added R23: 200k, Resistor_SMD:R_0603_1608Metric, F.Cu at (130.9, 112.4)
- added SW1: SW_SPST, Connector_PinHeader_2.54mm:PinHeader_1x02_P2.54mm_Horizontal, B.Cu at (121.3, 105.5)
- added U10: 74LVC1G32, Package_TO_SOT_SMD:SOT-23-5, F.Cu at (133.4, 96.8)
- added U11: 74LVC1G32, Package_TO_SOT_SMD:SOT-23-5, F.Cu at (136.9, 96.8)
- added U8: SN74LVC08ADRG3, Package_SO:SOIC-14_3.9x8.7mm_P1.27mm, F.Cu at (135.2, 105.2)
- added U9: NC7WZ14P6X, Package_TO_SOT_SMD:SOT-363_SC-70-6, F.Cu at (133.3, 112.4)
- J3: footprint Connector_PinHeader_2.54mm:PinHeader_1x02_P2.54mm_Horizontal -> Connector_PinHeader_2.54mm:PinHeader_1x02_P2.54mm_Vertical; moved to F.Cu
- turned J3 to 90 degrees
Connections:
- A1 pad 17: /EN_RELAY_DN -> /MCU_RELAY_DN
- A1 pad 18: /EN_RELAY_UP -> /MCU_RELAY_UP
- J11 pad 3: /EN_RELAY_DN -> /MCU_RELAY_DN
- J11 pad 4: /EN_RELAY_UP -> /MCU_RELAY_UP
- JP1 pad 1: +5V -> +3V3
Routing:
- net /MCU_RELAY_DN: track 0.00 -> 69.0 mm, vias 0 -> 2
- net /EN_RELAY_DN: track 86.4 -> 27.0 mm, vias 2 -> 0
- net /MCU_RELAY_UP: track 0.00 -> 58.6 mm, vias 0 -> 4
- net /EN_RELAY_UP: track 81.3 -> 24.3 mm, vias 2 -> 0
- net +5V: track 102.7 -> 45.7 mm, vias 4 -> 1
- net /BTN_DN: track 5.69 -> 55.9 mm, vias 0 -> 4
- net /BTN_UP: track 5.55 -> 55.3 mm, vias 0 -> 4
- net +3V3: track 72.9 -> 120.7 mm, vias 6 -> 7
- net /EN_MANUAL: track 0.00 -> 20.8 mm, vias 0 -> 1
- net Net-(U8-Pad3): track 0.00 -> 11.2 mm, vias 0 -> 2
- net Net-(U8-Pad11): track 0.00 -> 9.87 mm
- net Net-(U8-Pad4): track 0.00 -> 6.77 mm
- net Net-(U8-Pad6): track 0.00 -> 6.18 mm
- net Net-(U8-Pad1): track 0.00 -> 4.99 mm
- net /~{SW1}: track 55.7 -> 60.6 mm
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Other:
- board text added: "MAN"

Commit message: Hardware manual control option layout 2.
Parts:
- moved U11 16.7 mm to (120.5, 93.5), turned to 180 degrees
- moved U9 15.6 mm to (136.1, 97.1), turned to 90 degrees
- moved R23 13.9 mm to (136.1, 99.5), turned to 180 degrees
- moved U10 12.9 mm to (120.5, 97.0), turned to 180 degrees
- moved U8 11.8 mm to (128.9, 95.2), turned to -90 degrees
Routing:
- net /BTN_UP: track 55.3 -> 40.6 mm, vias 4 -> 2
- net /BTN_DN: track 55.9 -> 42.4 mm, vias 4 -> 2
- net /EN_RELAY_DN: track 27.0 -> 14.9 mm
- net /EN_RELAY_UP: track 24.3 -> 16.9 mm
- net /EN_MANUAL: track 20.8 -> 26.3 mm
- net /MCU_RELAY_DN: track 69.0 -> 63.7 mm
- net /MCU_RELAY_UP: track 58.6 -> 63.1 mm, vias 4 -> 2
- net +3V3: track 120.7 -> 119.8 mm, vias 7 -> 9

Commit message: Finish layout for hardware manual control option.
Routing:
- net +3V3: track 119.8 -> 158.6 mm, vias 9 -> 13
- net /BTN_DN: track 42.4 -> 63.9 mm, vias 2 -> 4
- net /BTN_UP: track 40.6 -> 56.3 mm, vias 2 -> 4
- net Net-(U8-Pad4): track 6.77 -> 13.2 mm
- net /MCU_RELAY_UP: track 63.1 -> 65.9 mm
- net /SRCK: track 70.0 -> 72.4 mm
- net /RCK: track 69.3 -> 71.7 mm
- net /MCU_RELAY_DN: track 63.7 -> 62.8 mm
- net Net-(U8-Pad1): track 4.99 -> 5.36 mm, vias 0 -> 2

Commit message: Add test point on manual enable and connect to MCU A1 pin.
Parts:
- added R24: 4k7, Resistor_SMD:R_0603_1608Metric, F.Cu at (167.7, 123.1)
- added TP4: TestPoint, TestPoint:TestPoint_THTPad_D1.5mm_Drill0.7mm, B.Cu at (135.2, 101.2)
Routing:
- net /EN_MANUAL: track 26.3 -> 93.2 mm, vias 1 -> 7
- net Net-(A1-Pad10): track 3.72 -> 10.9 mm, vias 0 -> 1

Commit message: 4 wires to up/down buttons: +12V, GND, UP input, DN input.
Move terminal block pin silkscreen labels away from edge.
Connections:
- J7 pad 1: /SW1EXT -> GND
- J7 pad 2: +12V -> /SW1EXT
- J7 pad 3: +12V -> /SW2EXT
- J7 pad 4: /SW2EXT -> +12V
Routing:
- net +12V: track 103.6 -> 96.6 mm, vias 3 -> 2
- net /SW1EXT: track 4.80 -> 8.58 mm
- net /SW2EXT: track 15.5 -> 12.5 mm

Commit message: Add board id & revision, reverse-polarity/unprotected warning on back.
Other:
- board text added: "Careful of reverse polarity, short-circuit. This board is not protected."
- board text added: "power-wedge-control, uno_r3 Rev 1"
Changed lines of the file:
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@@
     (property "Sheetname" "")
     (attr through_hole)
-    (fp_text reference "A1" (at 38.993 -25.348) (layer "B.SilkS")
+    (fp_text reference "A1" (at 39.201 -21.254) (layer "B.SilkS")
       (effects (font (size 0.6 0.6) (thickness 0.15)) (justify mirror))
     )
@@
     (effects (font (size 1.5 1.5) (thickness 0.3)) (justify right mirror))
   )
+  (gr_text "Careful of reverse polarity, short-circuit.\nThis board is not protected." (at 159.388 87.381) (layer "B.SilkS")
+    (effects (font (size 1.5 1.5) (thickness 0.3)) (justify mirror))
+  )
   (gr_text "6  7SegDisp  1" (at 143.2052 131.9276) (layer "B.SilkS")
     (effects (font (size 1.5 1.5) (thickness 0.3)) (justify mirror))
@@
     (effects (font (size 1.5 1.5) (thickness 0.3)) (justify right mirror))
   )
+  (gr_text "power-wedge-control, uno_r3\nRev 1" (at 190.088 101.681) (layer "B.SilkS")
+    (effects (font (size 1 1) (thickness 0.2)) (justify left mirror))
+  )
   (gr_text "Relays" (at 119.2038 130.2104) (layer "F.SilkS")

Commit message: Add board name, revision to front silkscreen and title block.
Extend 5V front filled zone.
Other:
- board text added: "Power Wedge Control"
- board text added: "Rev 1"
Changed lines of the file:
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@@
   )
   (paper "A4")
+  (title_block
+    (title "Power Wedge Control")
+    (date "2022-02-04")
+    (rev "1")
+  )
   (layers
     (0 "F.Cu" signal)
@@
     (effects (font (size 1.5 1.5) (thickness 0.3)))
   )
+  (gr_text "Rev 1" (at 187.638 109.481) (layer "F.SilkS")
+    (effects (font (size 1 1) (thickness 0.2)) (justify right))
+  )
+  (gr_text "Power Wedge\nControl" (at 187.688 105.031) (layer "F.SilkS")
+    (effects (font (size 2 2) (thickness 0.4)) (justify right))
+  )
   (gr_text "UP" (at 124.6844 127.6096 90) (layer "F.SilkS")
     (effects (font (size 1.5 1.5) (thickness 0.3)))
@@
         (xy 170.925 115.575)
         (xy 174.25 115.575)
+        (xy 174.231916 108.531144)
+        (xy 188.138 108.531)
+        (xy 188.138 83.581)
         (xy 174.15 76.625)
         (xy 190.75 76.625)
@@
     (polygon
       (pts
+        (xy 173.788 84.181)
+        (xy 187.688 84.181)
+        (xy 187.688 108.031)
+        (xy 173.8 108.031)
         (xy 173.8 115)
         (xy 170.8 115)

Commit message: Add 470 Ω resistor to limit current on +12V pin to up/down buttons.
Parts:
- added R25: 470, Resistor_SMD:R_0603_1608Metric, F.Cu at (168.2, 130.3)
Connections:
- J7 pad 4: +12V -> Net-(J7-Pad4)
Routing:
- net Net-(J7-Pad4): track 0.00 -> 4.63 mm
- net +12V: track 96.6 -> 92.3 mm
Changed lines of the file:
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@@
   (net 80 "Net-(U10-Pad1)")
   (net 81 "Net-(U11-Pad1)")
+  (net 82 "Net-(J7-Pad4)")
   (footprint "TerminalBlock_Phoenix:TerminalBlock_Phoenix_PT-1,5-2-3.5-H_1x02_P3.50mm_Horizontal" (layer "F.Cu")
     (at 126.9088 134.6554)
@@
     )
   )
+  (footprint "Resistor_SMD:R_0603_1608Metric" (layer "F.Cu")
+    (at 168.188 130.331 180)
+    (descr "Resistor SMD 0603 (1608 Metric), square (rectangular) end terminal, IPC_7351 nominal, (Body size source: IPC-SM-782 page 72, https://www.pcb-3d.com/wordpress/wp-content/uploads/ipc-sm-782a_amendment_1_and_2.pdf), generated with kicad-footprint-generator")
+    (tags "resistor")
+    (property "Sheetfile" "power-wedge-control.kicad_sch")
+    (property "Sheetname" "")
+    (attr smd)
+    (fp_text reference "R25" (at 0 -1.43) (layer "F.SilkS")
+      (effects (font (size 0.6 0.6) (thickness 0.15)))
+    )
+    (fp_text value "470" (at 0 1.43) (layer "F.Fab")
+      (effects (font (size 1 1) (thickness 0.15)))
+    )
+    (fp_text user "${REFERENCE}" (at 0 0) (layer "F.Fab")
+      (effects (font (size 0.6 0.6) (thickness 0.06)))
+    )
+    (fp_line (start -0.237258 0.5225) (end 0.237258 0.5225) (layer "F.SilkS") (width 0.12))
+    (fp_line (start -0.237258 -0.5225) (end 0.237258 -0.5225) (layer "F.SilkS") (width 0.12))
+    (fp_line (start -1.48 0.73) (end -1.48 -0.73) (layer "F.CrtYd") (width 0.05))
+    (fp_line (start -1.48 -0.73) (end 1.48 -0.73) (layer "F.CrtYd") (width 0.05))
+    (fp_line (start 1.48 -0.73) (end 1.48 0.73) (layer "F.CrtYd") (width 0.05))
+    (fp_line (start 1.48 0.73) (end -1.48 0.73) (layer "F.CrtYd") (width 0.05))
+    (fp_line (start 0.8 -0.4125) (end 0.8 0.4125) (layer "F.Fab") (width 0.1))
+    (fp_line (start -0.8 0.4125) (end -0.8 -0.4125) (layer "F.Fab") (width 0.1))
+    (fp_line (start -0.8 -0.4125) (end 0.8 -0.4125) (layer "F.Fab") (width 0.1))
+    (fp_line (start 0.8 0.4125) (end -0.8 0.4125) (layer "F.Fab") (width 0.1))
+    (pad "1" smd roundrect (at -0.825 0 180) (size 0.8 0.95) (layers "F.Cu" "F.Paste" "F.Mask") (roundrect_rratio 0.25)
+      (net 4 "+12V") (pintype "passive"))
+    (pad "2" smd roundrect (at 0.825 0 180) (size 0.8 0.95) (layers "F.Cu" "F.Paste" "F.Mask") (roundrect_rratio 0.25)
+      (net 82 "Net-(J7-Pad4)") (pintype "passive"))
+    (model "${KICAD6_3DMODEL_DIR}/Resistor_SMD.3dshapes/R_0603_1608Metric.wrl"
+      (offset (xyz 0 0 0))
+      (scale (xyz 1 1 1))
+      (rotate (xyz 0 0 0))
+    )
+  )
   (footprint "Capacitor_SMD:C_0603_1608Metric" (layer "F.Cu")
     (at 179.9336 130.2512)
@@
       (net 70 "/SW2EXT") (pinfunction "Pin_3") (pintype "passive"))
     (pad "4" thru_hole circle locked (at 10.5 0) (size 2.4 2.4) (drill 1.2) (layers *.Cu *.Mask)
-      (net 4 "+12V") (pinfunction "Pin_4") (pintype "passive"))
+      (net 82 "Net-(J7-Pad4)") (pinfunction "Pin_4") (pintype "passive"))
     (model "${KICAD6_3DMODEL_DIR}/TerminalBlock_Phoenix.3dshapes/TerminalBlock_Phoenix_PT-1,5-4-3.5-H_1x04_P3.50mm_Horizontal.wrl"
       (offset (xyz 0 0 0))
@@
   (segment (start 115.8224 124.8664) (end 115.8224 123.4668) (width 0.8) (layer "F.Cu") (net 3))
   (segment (start 153 124.5) (end 154.138 124.5) (width 0.8) (layer "F.Cu") (net 4))
+  (segment (start 169.013 130.331) (end 169.013 129.456) (width 0.8) (layer "F.Cu") (net 4))
   (segment (start 154.9562 115.9502) (end 155.6562 115.2502) (width 0.8) (layer "F.Cu") (net 4))
   (segment (start 119.198 120.4346) (end 119.198 119.0244) (width 0.8) (layer "F.Cu") (net 4))
@@
   (segment (start 154.138 124.5) (end 166 124.5) (width 0.8) (layer "F.Cu") (net 4))
   (segment (start 153.421 115.9502) (end 153.421 124.079) (width 0.8) (layer "F.Cu") (net 4))
-  (segment (start 167.767 129.7178) (end 166.6136 130.8712) (width 0.8) (layer "F.Cu") (net 4))
   (segment (start 127.741518 124.499118) (end 126.9088 125.331836) (width 0.8) (layer "F.Cu") (net 4))
   (segment (start 154.138 124.5) (end 153.842 124.5) (width 0.8) (layer "F.Cu") (net 4))
-  (segment (start 166.6136 130.8712) (end 166.6136 134.6554) (width 0.8) (layer "F.Cu") (net 4))
   (segment (start 126.119 120.4346) (end 126.6656 119.888) (width 0.8) (layer "F.Cu") (net 4))
   (segment (start 132.650482 124.499118) (end 132.6878 124.4618) (width 0.8) (layer "F.Cu") (net 4))
@@
   (segment (start 122.566 119.0092) (end 122.6524 118.9228) (width 0.8) (layer "F.Cu") (net 4))
   (segment (start 126.9088 125.331836) (end 126.9088 134.6554) (width 0.8) (layer "F.Cu") (net 4))
-  (segment (start 167.767 127.635) (end 167.767 129.7178) (width 0.8) (layer "F.Cu") (net 4))
   (segment (start 147.8788 124.5) (end 153 124.5) (width 0.8) (layer "F.Cu") (net 4))
   (segment (start 126.056 120.4346) (end 126.119 120.4346) (width 0.8) (layer "F.Cu") (net 4))
@@
   (segment (start 155.6562 115.2502) (end 155.6562 116.3832) (width 0.8) (layer "F.Cu") (net 4))
   (segment (start 116.5056 118.9228) (end 119.0964 118.9228) (width 0.8) (layer "F.Cu") (net 4))
+  (segment (start 169.013 129.456) (end 167.767 128.21) (width 0.8) (layer "F.Cu") (net 4))
   (segment (start 115.708 120.7562) (end 115.708 119.7204) (width 0.8) (layer "F.Cu") (net 4))
   (segment (start 125.7004 118.9228) (end 126.6656 119.888) (width 0.8) (layer "F.Cu") (net 4))
   (segment (start 153.842 124.5) (end 153.421 124.079) (width 0.8) (layer "F.Cu") (net 4))
   (segment (start 153.421 124.079) (end 153 124.5) (width 0.8) (layer "F.Cu") (net 4))
+  (segment (start 167.767 128.21) (end 167.767 127.635) (width 0.8) (layer "F.Cu") (net 4))
   (segment (start 142.388 124.481) (end 132.650482 124.499118) (width 0.8) (layer "F.Cu") (net 4))
   (via (at 147.8788 124.5) (size 1.6) (drill 0.8) (layers "F.Cu" "B.Cu") (net 4))
@@
   (segment (start 128.239519 94.874519) (end 128.89 95.525) (width 0.3) (layer "F.Cu") (net 81))
   (segment (start 128.89 95.525) (end 128.89 97.7) (width 0.3) (layer "F.Cu") (net 81))
+  (segment (start 167.363 130.331) (end 167.363 131.006) (width 0.4) (layer "F.Cu") (net 82))
+  (segment (start 167.363 131.006) (end 166.6136 131.7554) (width 0.4) (layer "F.Cu") (net 82))
+  (segment (start 166.6136 131.7554) (end 166.6136 134.6554) (width 0.4) (layer "F.Cu") (net 82))
   (zone (net 0) (net_name "") (layer "F.Cu") (hatch edge 0.508)
     (connect_pads (clearance 0))
