File: power-wedge-control.kicad_sch (KiCad schematic)
At the start: 32 parts, among them J1 Conn_01x02, J2 Conn_01x03, J3 Conn_01x02, J4 Conn_01x03, J5 Conn_01x03, Q1 MMBT3904L, Q2 DMP3099L, Q3 MMBT3904L, Q4 DMP3099L, U1 LM7805_TO220

Commit message: WIP. Add relay LEDs, ui/display connection.
Parts:
- added D3, D4: LED, LED_SMD:LED_0603_1608Metric, symbol Device:LED
- added J6: Conn_01x06_Female, Connector_PinHeader_2.54mm:PinHeader_1x06_P2.54mm_Vertical, symbol Connector:Conn_01x06_Female
- added R10, R9: 1k, Resistor_SMD:R_0603_1608Metric, symbol Device:R
Connections:
- net +5V: now also J6.6 (Pin_6)
- net GND: now also D3.1 (K), D4.1 (K), J6.1 (Pin_1)
- net RELAY_DN+: now also R10.2
- net RELAY_UP+: now also R9.2
- new net: D3.2 (A), R9.1
- new net: D4.2 (A), R10.1
- new net CLK: J6.4 (Pin_4)
- new net LE: J6.3 (Pin_3)
- new net OE: J6.5 (Pin_5)
- new net SDI: J6.2 (Pin_2)
Other:
- note added: "5V Regulated Power Supply"
- note added: "LED Display Connection"
- note added: "TODO: Board id & revision on back/front."
- note added: "TODO: Do we need 3V3? Or does Huzzah32 Feather make 3.3V?"
- moved on the sheet: D1, D2, J2

Commit message: Add output enable, MCU wants relay up/down green LEDs.
Parts:
- added JP1: Jumper_2_Open, Connector_PinHeader_2.54mm:PinHeader_1x02_P2.54mm_Vertical, symbol Jumper:Jumper_2_Open
- added JP2, JP3: Jumper_2_Bridged, Jumper:SolderJumper-2_P1.3mm_Bridged_RoundedPad1.0x1.5mm, symbol Jumper:Jumper_2_Bridged
- added LED3, LED4: LED_GRN, LED_SMD:LED_0603_1608Metric, symbol Device:LED
- added Q5, Q6: MMBT3904L, Package_TO_SOT_SMD:SOT-23, symbol Device:Q_NPN_BEC
- added R11, R12: 10k, Resistor_SMD:R_0603_1608Metric, symbol Device:R
- added R13, R14: 1k, Resistor_SMD:R_0603_1608Metric, symbol Device:R
- renumbered D3 to LED1, D4 to LED2
Connections:
- net +5V: now also JP1.1 (A), JP2.1 (A), JP3.1 (A); no longer J4.3 (Pin_3), J5.3 (Pin_3), J6.6 (Pin_6)
- net EN_RELAY_DN: now also R14.2
- net EN_RELAY_UP: now also R13.2
- net GND: now also LED3.1 (K), LED4.1 (K)
- net at R2.2: now also Q6.3 (C); no longer Q1.3 (C)
- net at R5.2: now also Q5.3 (C); no longer Q3.3 (C)
- new net: Q1.3 (C), Q6.2 (E)
- new net: Q3.3 (C), Q5.2 (E)
- new net: Q6.1 (B), R12.1
- new net: LED3.2 (A), R13.1
- new net: Q5.1 (B), R11.1
- new net: LED4.2 (A), R14.1
- new net EN_OUTPUT: JP1.2 (B), R11.2, R12.2
- new net SENS_PWR: J4.3 (Pin_3), J5.3 (Pin_3), JP3.2 (B)
- new net UI_PWR: J6.6 (Pin_6), JP2.2 (B)
Other:
- note added: "TODO: Add UP/DN dash buttons (w/hardware debounce)"
- note added: "TODO: Invert output_enable to output_disable?"
- note added: "TODO: Test points, pins, or jumpers for accessing key circuits?"
- note added: "Test point and LED indicators"
- moved on the sheet: C1, C2, C3, C4, D1, D2, J1, J2, J3, J4, J5, L1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

Commit message: Swap CLK and LE pins on LED UI display connection.
Connections:
- net CLK: now also J6.3 (Pin_3); no longer J6.4 (Pin_4)
- net LE: now also J6.4 (Pin_4); no longer J6.3 (Pin_3)
- net UI_PWR renamed UI_VDD
Changed lines of the file:
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@@
     (stroke (width 0) (type default) (color 0 0 0 0))
   )
-  (wire (pts (xy 245.11 41.91) (xy 252.73 41.91))
+  (wire (pts (xy 246.38 36.83) (xy 254 36.83))
     (stroke (width 0) (type default) (color 0 0 0 0))
   )
@@
     (stroke (width 0) (type default) (color 0 0 0 0))
   )
+  (wire (pts (xy 246.38 44.45) (xy 254 44.45))
+    (stroke (width 0) (type default) (color 0 0 0 0))
+  )
   (wire (pts (xy 147.32 132.08) (xy 147.32 139.7))
     (stroke (width 0) (type default) (color 0 0 0 0))
@@
     (stroke (width 0) (type default) (color 0 0 0 0))
   )
-  (wire (pts (xy 245.11 34.29) (xy 252.73 34.29))
-    (stroke (width 0) (type default) (color 0 0 0 0))
-  )
   (wire (pts (xy 120.65 83.82) (xy 177.8 83.82))
     (stroke (width 0) (type default) (color 0 0 0 0))
@@
     (stroke (width 0) (type default) (color 0 0 0 0))
   )
+  (wire (pts (xy 246.38 46.99) (xy 254 46.99))
+    (stroke (width 0) (type default) (color 0 0 0 0))
+  )
   (wire (pts (xy 133.35 55.88) (xy 148.59 55.88))
     (stroke (width 0) (type default) (color 0 0 0 0))
@@
     (stroke (width 0) (type default) (color 0 0 0 0))
   )
-  (wire (pts (xy 245.11 46.99) (xy 252.73 46.99))
+  (wire (pts (xy 246.38 41.91) (xy 254 41.91))
     (stroke (width 0) (type default) (color 0 0 0 0))
   )
@@
     (stroke (width 0) (type default) (color 0 0 0 0))
   )
-  (wire (pts (xy 245.11 39.37) (xy 252.73 39.37))
-    (stroke (width 0) (type default) (color 0 0 0 0))
-  )
   (wire (pts (xy 143.51 189.23) (xy 143.51 193.04))
     (stroke (width 0) (type default) (color 0 0 0 0))
   )
+  (wire (pts (xy 246.38 39.37) (xy 254 39.37))
+    (stroke (width 0) (type default) (color 0 0 0 0))
+  )
   (wire (pts (xy 82.55 191.77) (xy 96.52 191.77))
     (stroke (width 0) (type default) (color 0 0 0 0))
@@
     (stroke (width 0) (type default) (color 0 0 0 0))
   )
+  (wire (pts (xy 246.38 34.29) (xy 254 34.29))
+    (stroke (width 0) (type default) (color 0 0 0 0))
+  )
   (wire (pts (xy 114.3 185.42) (xy 114.3 187.96))
     (stroke (width 0) (type default) (color 0 0 0 0))
@@
     (stroke (width 0) (type default) (color 0 0 0 0))
   )
-  (wire (pts (xy 245.11 36.83) (xy 252.73 36.83))
-    (stroke (width 0) (type default) (color 0 0 0 0))
-  )
   (wire (pts (xy 68.58 184.15) (xy 82.55 184.15))
     (stroke (width 0) (type default) (color 0 0 0 0))
   )
   (wire (pts (xy 40.64 162.56) (xy 27.94 162.56))
-    (stroke (width 0) (type default) (color 0 0 0 0))
-  )
-  (wire (pts (xy 245.11 44.45) (xy 252.73 44.45))
     (stroke (width 0) (type default) (color 0 0 0 0))
   )
@@
     (effects (font (size 1.27 1.27)) (justify left bottom))
   )
-  (label "CLK" (at 252.73 39.37 180)
-    (effects (font (size 1.27 1.27)) (justify right bottom))
-  )
-  (label "UI_PWR" (at 252.73 34.29 180)
+  (label "UI_VDD" (at 254 34.29 180)
     (effects (font (size 1.27 1.27)) (justify right bottom))
   )
@@
     (effects (font (size 1.27 1.27)) (justify left bottom))
   )
-  (label "GND" (at 252.73 46.99 180)
-    (effects (font (size 1.27 1.27)) (justify right bottom))
-  )
   (label "GND" (at 40.64 191.77 180)
     (effects (font (size 1.27 1.27)) (justify right bottom))
@@
     (effects (font (size 1.27 1.27)) (justify left bottom))
   )
+  (label "LE" (at 254 39.37 180)
+    (effects (font (size 1.27 1.27)) (justify right bottom))
+  )
   (label "EN_OUTPUT" (at 266.7 67.31 180)
     (effects (font (size 1.27 1.27)) (justify right bottom))
@@
     (effects (font (size 1.27 1.27)) (justify right bottom))
   )
+  (label "CLK" (at 254 41.91 180)
+    (effects (font (size 1.27 1.27)) (justify right bottom))
+  )
+  (label "SDI" (at 254 44.45 180)
+    (effects (font (size 1.27 1.27)) (justify right bottom))
+  )
   (label "SENS_PWR" (at 40.64 162.56 180)
     (effects (font (size 1.27 1.27)) (justify right bottom))
@@
     (effects (font (size 1.27 1.27)) (justify right bottom))
   )
+  (label "OE" (at 254 36.83 180)
+    (effects (font (size 1.27 1.27)) (justify right bottom))
+  )
   (label "ANGL2" (at 40.64 184.15 180)
     (effects (font (size 1.27 1.27)) (justify right bottom))
   )
+  (label "GND" (at 254 46.99 180)
+    (effects (font (size 1.27 1.27)) (justify right bottom))
+  )
   (label "EN_RELAY_DN" (at 125.73 193.04 180)
     (effects (font (size 1.27 1.27)) (justify right bottom))
@@
     (effects (font (size 1.27 1.27)) (justify right bottom))
   )
-  (label "LE" (at 252.73 41.91 180)
-    (effects (font (size 1.27 1.27)) (justify right bottom))
-  )
   (label "ANGL2_REF5V" (at 148.59 58.42 180)
     (effects (font (size 1.27 1.27)) (justify right bottom))
   )
-  (label "UI_PWR" (at 266.7 72.39 180)
-    (effects (font (size 1.27 1.27)) (justify right bottom))
-  )
-  (label "SDI" (at 252.73 44.45 180)
-    (effects (font (size 1.27 1.27)) (justify right bottom))
-  )
-  (label "OE" (at 252.73 36.83 180)
+  (label "UI_VDD" (at 266.7 72.39 180)
     (effects (font (size 1.27 1.27)) (justify right bottom))
   )
@@
     (pin "2")
   )
-  (symbol (lib_id "Connector:Conn_01x06_Female") (at 240.03 41.91 180) (unit 1)
-    (in_bom yes) (on_board yes)
-    (property "Reference" "J6" (id 0) (at 242.57 48.26 0))
-    (property "Value" "Conn_01x06_Female" (id 1) (at 238.76 40.64 90))
-    (property "Footprint" "Connector_PinHeader_2.54mm:PinHeader_1x06_P2.54mm_Vertical" (id 2) (at 240.03 41.91 0)
-      (effects (font (size 1.27 1.27)) hide)
-    )
-    (property "Datasheet" "~" (id 3) (at 240.03 41.91 0)
+  (symbol (lib_id "power:+5V") (at 80.01 26.67 270) (unit 1)
+    (in_bom yes) (on_board yes) (fields_autoplaced)
+    (property "Reference" "#PWR011" (id 0) (at 76.2 26.67 0)
+      (effects (font (size 1.27 1.27)) hide)
+    )
+    (property "Value" "+5V" (id 1) (at 83.82 26.6699 90)
+      (effects (font (size 1.27 1.27)) (justify left))
+    )
+    (property "Footprint" "" (id 2) (at 80.01 26.67 0)
+      (effects (font (size 1.27 1.27)) hide)
+    )
+    (property "Datasheet" "" (id 3) (at 80.01 26.67 0)
+      (effects (font (size 1.27 1.27)) hide)
+    )
+    (pin "1")
+  )
+  (symbol (lib_id "Device:LED") (at 160.02 160.02 270) (unit 1)
+    (in_bom yes) (on_board yes)
+    (property "Reference" "LED1" (id 0) (at 157.48 160.02 0)
+      (effects (font (size 1.27 1.27)) (justify left))
+    )
+    (property "Value" "LED" (id 1) (at 162.56 158.75 0)
+      (effects (font (size 1.27 1.27)) (justify left))
+    )
+    (property "Footprint" "LED_SMD:LED_0603_1608Metric" (id 2) (at 160.02 160.02 0)
+      (effects (font (size 1.27 1.27)) hide)
+    )
+    (property "Datasheet" "~" (id 3) (at 160.02 160.02 0)
+      (effects (font (size 1.27 1.27)) hide)
+    )
+    (pin "1")
+    (pin "2")
+  )
+  (symbol (lib_id "Connector:Conn_01x06_Female") (at 241.3 41.91 180) (unit 1)
+    (in_bom yes) (on_board yes)
+    (property "Reference" "J6" (id 0) (at 243.84 48.26 0))
+    (property "Value" "Conn_01x06_Female" (id 1) (at 240.03 40.64 90))
+    (property "Footprint" "Connector_PinHeader_2.54mm:PinHeader_1x06_P2.54mm_Vertical" (id 2) (at 241.3 41.91 0)
+      (effects (font (size 1.27 1.27)) hide)
+    )
+    (property "Datasheet" "~" (id 3) (at 241.3 41.91 0)
       (effects (font (size 1.27 1.27)) hide)
     )
@@
     (pin "6")
   )
-  (symbol (lib_id "power:+5V") (at 80.01 26.67 270) (unit 1)
-    (in_bom yes) (on_board yes) (fields_autoplaced)
-    (property "Reference" "#PWR011" (id 0) (at 76.2 26.67 0)
-      (effects (font (size 1.27 1.27)) hide)
-    )
-    (property "Value" "+5V" (id 1) (at 83.82 26.6699 90)
-      (effects (font (size 1.27 1.27)) (justify left))
-    )
-    (property "Footprint" "" (id 2) (at 80.01 26.67 0)
-      (effects (font (size 1.27 1.27)) hide)
-    )
-    (property "Datasheet" "" (id 3) (at 80.01 26.67 0)
-      (effects (font (size 1.27 1.27)) hide)
-    )
-    (pin "1")
-  )
-  (symbol (lib_id "Device:LED") (at 160.02 160.02 270) (unit 1)
-    (in_bom yes) (on_board yes)
-    (property "Reference" "LED1" (id 0) (at 157.48 160.02 0)
-      (effects (font (size 1.27 1.27)) (justify left))
-    )
-    (property "Value" "LED" (id 1) (at 162.56 158.75 0)
-      (effects (font (size 1.27 1.27)) (justify left))
-    )
-    (property "Footprint" "LED_SMD:LED_0603_1608Metric" (id 2) (at 160.02 160.02 0)
-      (effects (font (size 1.27 1.27)) hide)
-    )
-    (property "Datasheet" "~" (id 3) (at 160.02 160.02 0)
-      (effects (font (size 1.27 1.27)) hide)
-    )
-    (pin "1")
-    (pin "2")
-  )
   (symbol (lib_id "power:+12V") (at 118.11 25.4 0) (unit 1)
     (in_bom yes) (on_board yes)
@@
       (reference "J5") (unit 1) (value "Conn_01x03") (footprint "TerminalBlock_Phoenix:TerminalBlock_Phoenix_PT-1,5-3-3.5-H_1x03_P3.50mm_Horizontal")
     )
-    (path "/a70e11b4-d908-421b-920d-a8abf0b3eac7"
+    (path "/c5c924a2-bc0e-4c14-adc4-fe078f64fb1f"
       (reference "J6") (unit 1) (value "Conn_01x06_Female") (footprint "Connector_PinHeader_2.54mm:PinHeader_1x06_P2.54mm_Vertical")
     )

Commit message: Add Up/Down buttons switch input with hardware debounce.
HW debounce copied from ultrasonic PCB project.
Parts:
- added J7: Conn_01x04_Female, TerminalBlock_Phoenix:TerminalBlock_Phoenix_PT-1,5-4-3.5-H_1x04_P3.50mm_Horizontal, symbol Connector:Conn_01x04_Female
- added JP3: Jumper_2_Bridged, Jumper:SolderJumper-2_P1.3mm_Bridged_RoundedPad1.0x1.5mm, symbol Jumper:Jumper_2_Bridged
- J6: footprint Connector_PinHeader_2.54mm:PinHeader_1x06_P2.54mm_Vertical -> TerminalBlock_Phoenix:TerminalBlock_Phoenix_PT-1,5-6-3.5-H_1x06_P3.50mm_Horizontal
- renumbered JP3 to JP4
Connections:
- net +5V: now also JP3.1 (A)
- net BTN_DN: now reaches A1.17 (D2)
- net BTN_UP: now reaches A1.18 (D3)
- net UI_VDD renamed UI_PWR
- new net BTN_PWR: JP3.2 (B)
- new net HWDebounce/SW1IN: J7.1 (Pin_1)
- new net HWDebounce/SW2IN: J7.4 (Pin_4)
- new net HWDebounce/SWGND: J7.2 (Pin_2), J7.3 (Pin_3)
- no-connect marks 49 -> 47
Other:
- added sheet HWDebounce (hw-debounce.kicad_sch)
- note added: "LED UI Display Connection"
- note added: "Power Input"
- note added: "TODO: Button (hardware) debounce timing/tuning."
- note added: "TODO: Power input peripherals via MCU VCC regulator vs external VCC reg?"
- note added: "Up/Down Buttons"
- note removed: "LED Display Connection"
- moved on the sheet: J1, J6, JP4

Commit message: Fix hardware debounce circuit (was incorrect).
Connections:
- net HWDebounce/SWGND is gone; now on net GND: J7.2 (Pin_2), J7.3 (Pin_3)
Other:
- sheet HWDebounce ports: added none; removed SWGND
Changed lines of the file:
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@@
-    (stroke (width 0) (type default) (color 0 0 0 0))
-  )
-  (wire (pts (xy 43.18 102.87) (xy 43.18 100.33))
     (stroke (width 0) (type default) (color 0 0 0 0))
   )
@@
   )
   (label "EN_RELAY_UP" (at 106.68 154.94 0)
+    (effects (font (size 1.27 1.27)) (justify left bottom))
+  )
+  (label "GND" (at 26.67 91.44 0)
     (effects (font (size 1.27 1.27)) (justify left bottom))
   )
@@
     (pin "2")
   )
-  (symbol (lib_id "power:GND") (at 43.18 102.87 0) (unit 1)
-    (in_bom yes) (on_board yes)
-    (property "Reference" "#PWR016" (id 0) (at 43.18 109.22 0)
-      (effects (font (size 1.27 1.27)) hide)
-    )
-    (property "Value" "GND" (id 1) (at 43.307 106.1212 90)
-      (effects (font (size 1.27 1.27)) (justify right))
-    )
-    (property "Footprint" "" (id 2) (at 43.18 102.87 0)
-      (effects (font (size 1.27 1.27)) hide)
-    )
-    (property "Datasheet" "" (id 3) (at 43.18 102.87 0)
-      (effects (font (size 1.27 1.27)) hide)
-    )
-    (pin "1")
-  )
   (symbol (lib_id "Device:C") (at 33.02 30.48 0) (unit 1)
     (in_bom yes) (on_board yes)
@@
       (effects (font (size 1.27 1.27)) (justify left top))
     )
-    (pin "SWGND" bidirectional (at 33.02 91.44 180)
-      (effects (font (size 1.27 1.27)) (justify left))
-    )
     (pin "SW1IN" bidirectional (at 33.02 88.9 180)
       (effects (font (size 1.27 1.27)) (justify left))
@@
       (effects (font (size 1.27 1.27)) (justify right))
     )
-    (pin "GND" bidirectional (at 43.18 100.33 270)
+    (pin "GND" bidirectional (at 33.02 91.44 180)
       (effects (font (size 1.27 1.27)) (justify left))
     )
@@
       (reference "#PWR015") (unit 1) (value "GND") (footprint "")
     )
-    (path "/4370dc21-ae67-473b-be84-47ac990c560d"
-      (reference "#PWR016") (unit 1) (value "GND") (footprint "")
-    )
     (path "/fd5920d6-c9a8-4baf-80de-0fa06e4ffab0"

Commit message: Connect LED UI display connector to MCU pins.
Connections:
- net CLK: now also A1.21 (D6)
- net LE: now also A1.20 (D5)
- net OE: now also A1.19 (D4)
- net SDI: now also A1.22 (D7)
- no-connect marks 47 -> 43
Changed lines of the file:
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@@
   (no_connect (at 123.19 25.4))
   (no_connect (at 107.95 35.56))
-  (no_connect (at 107.95 45.72))
-  (no_connect (at 107.95 48.26))
-  (no_connect (at 107.95 50.8))
-  (no_connect (at 107.95 53.34))
   (no_connect (at 107.95 55.88))
   (no_connect (at 107.95 58.42))
@@
     (stroke (width 0) (type default) (color 0 0 0 0))
   )
+  (wire (pts (xy 92.71 48.26) (xy 107.95 48.26))
+    (stroke (width 0) (type default) (color 0 0 0 0))
+  )
   (wire (pts (xy 241.3 82.55) (xy 245.11 82.55))
     (stroke (width 0) (type default) (color 0 0 0 0))
@@
     (stroke (width 0) (type default) (color 0 0 0 0))
   )
+  (wire (pts (xy 92.71 50.8) (xy 107.95 50.8))
+    (stroke (width 0) (type default) (color 0 0 0 0))
+  )
   (wire (pts (xy 172.72 102.87) (xy 172.72 100.33))
     (stroke (width 0) (type default) (color 0 0 0 0))
@@
     (stroke (width 0) (type default) (color 0 0 0 0))
   )
+  (wire (pts (xy 92.71 45.72) (xy 107.95 45.72))
+    (stroke (width 0) (type default) (color 0 0 0 0))
+  )
   (wire (pts (xy 49.53 34.29) (xy 62.23 34.29))
     (stroke (width 0) (type default) (color 0 0 0 0))
@@
   )
   (wire (pts (xy 120.65 78.74) (xy 123.19 78.74))
+    (stroke (width 0) (type default) (color 0 0 0 0))
+  )
+  (wire (pts (xy 92.71 53.34) (xy 107.95 53.34))
     (stroke (width 0) (type default) (color 0 0 0 0))
   )
@@
     (effects (font (size 1.27 1.27)) (justify left bottom))
   )
+  (label "CLK" (at 92.71 50.8 0)
+    (effects (font (size 1.27 1.27)) (justify left bottom))
+  )
   (label "EN_OUTPUT" (at 106.68 113.03 0)
     (effects (font (size 1.27 1.27)) (justify left bottom))
@@
     (effects (font (size 1.27 1.27)) (justify left bottom))
   )
+  (label "LE" (at 92.71 48.26 0)
+    (effects (font (size 1.27 1.27)) (justify left bottom))
+  )
   (label "EN_RELAY_UP" (at 92.71 63.5 0)
     (effects (font (size 1.27 1.27)) (justify left bottom))
@@
     (effects (font (size 1.27 1.27)) (justify right bottom))
   )
+  (label "SDI" (at 92.71 53.34 0)
+    (effects (font (size 1.27 1.27)) (justify left bottom))
+  )
   (label "ANGL2_REF5V" (at 148.59 58.42 180)
     (effects (font (size 1.27 1.27)) (justify right bottom))
@@
     (effects (font (size 1.27 1.27)) (justify right bottom))
   )
+  (label "OE" (at 92.71 45.72 0)
+    (effects (font (size 1.27 1.27)) (justify left bottom))
+  )
   (symbol (lib_id "Connector_Generic:Conn_01x02") (at 22.86 58.42 0) (mirror y) (unit 1)

Commit message: Route remaining traces (relay control, 5V).
Silkscreen clean up.
Parts:
- J3, JP1: footprint Connector_PinHeader_2.54mm:PinHeader_1x02_P2.54mm_Vertical -> Connector_PinHeader_2.54mm:PinHeader_1x02_P2.54mm_Horizontal
Changed lines of the file:
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@@
     (property "Reference" "J3" (id 0) (at 109.22 185.42 0))
     (property "Value" "Conn_01x02" (id 1) (at 106.68 189.23 90))
-    (property "Footprint" "Connector_PinHeader_2.54mm:PinHeader_1x02_P2.54mm_Vertical" (id 2) (at 109.22 187.96 0)
+    (property "Footprint" "Connector_PinHeader_2.54mm:PinHeader_1x02_P2.54mm_Horizontal" (id 2) (at 109.22 187.96 0)
       (effects (font (size 1.27 1.27)) hide)
     )
@@
       (effects (font (size 1.27 1.27)) hide)
     )
-    (property "Footprint" "Connector_PinHeader_2.54mm:PinHeader_1x02_P2.54mm_Vertical" (id 2) (at 250.19 67.31 0)
+    (property "Footprint" "Connector_PinHeader_2.54mm:PinHeader_1x02_P2.54mm_Horizontal" (id 2) (at 250.19 67.31 0)
       (effects (font (size 1.27 1.27)) hide)
     )
@@
     )
     (path "/00000000-0000-0000-0000-000061ace482"
-      (reference "J3") (unit 1) (value "Conn_01x02") (footprint "Connector_PinHeader_2.54mm:PinHeader_1x02_P2.54mm_Vertical")
+      (reference "J3") (unit 1) (value "Conn_01x02") (footprint "Connector_PinHeader_2.54mm:PinHeader_1x02_P2.54mm_Horizontal")
     )
     (path "/00000000-0000-0000-0000-000061a46160"
@@
     )
     (path "/e2be7400-dc56-4426-9ef7-bf338a64a34d"
-      (reference "JP1") (unit 1) (value "Jumper_2_Open") (footprint "Connector_PinHeader_2.54mm:PinHeader_1x02_P2.54mm_Vertical")
+      (reference "JP1") (unit 1) (value "Jumper_2_Open") (footprint "Connector_PinHeader_2.54mm:PinHeader_1x02_P2.54mm_Horizontal")
     )
     (path "/0caf6566-794a-4113-b149-e2d9cc5f313e"

Commit message: 100n on sensor power. Connector silkscreen labels larger (1.5mm)
Parts:
- added C13: 100n, Capacitor_SMD:C_0603_1608Metric, symbol Device:C
Connections:
- net GND: now also C13.2
- net SENS_PWR: now also C13.1
Changed lines of the file:
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@@
   (junction (at 68.58 191.77) (diameter 0) (color 0 0 0 0)
   )
+  (junction (at 269.24 82.55) (diameter 0) (color 0 0 0 0)
+  )
   (junction (at 154.94 132.08) (diameter 0) (color 0 0 0 0)
   )
@@
   )
   (junction (at 21.59 34.29) (diameter 0) (color 0 0 0 0)
+  )
+  (junction (at 269.24 90.17) (diameter 0) (color 0 0 0 0)
   )
   (junction (at 165.1 107.95) (diameter 0) (color 0 0 0 0)
@@
     (stroke (width 0) (type default) (color 0 0 0 0))
   )
+  (wire (pts (xy 262.89 90.17) (xy 269.24 90.17))
+    (stroke (width 0) (type default) (color 0 0 0 0))
+  )
   (wire (pts (xy 133.35 55.88) (xy 148.59 55.88))
     (stroke (width 0) (type default) (color 0 0 0 0))
   )
+  (wire (pts (xy 269.24 82.55) (xy 271.78 82.55))
+    (stroke (width 0) (type default) (color 0 0 0 0))
+  )
   (wire (pts (xy 120.65 113.03) (xy 120.65 144.78))
     (stroke (width 0) (type default) (color 0 0 0 0))
@@
     (stroke (width 0) (type default) (color 0 0 0 0))
   )
+  (wire (pts (xy 269.24 90.17) (xy 271.78 90.17))
+    (stroke (width 0) (type default) (color 0 0 0 0))
+  )
   (wire (pts (xy 33.02 60.96) (xy 27.94 60.96))
     (stroke (width 0) (type default) (color 0 0 0 0))
@@
     (stroke (width 0) (type default) (color 0 0 0 0))
   )
-  (wire (pts (xy 255.27 82.55) (xy 266.7 82.55))
+  (wire (pts (xy 255.27 82.55) (xy 269.24 82.55))
     (stroke (width 0) (type default) (color 0 0 0 0))
   )
@@
   (label "SENS_PWR" (at 266.7 82.55 180)
     (effects (font (size 1.27 1.27)) (justify right bottom))
+  )
+  (label "GND" (at 262.89 90.17 0)
+    (effects (font (size 1.27 1.27)) (justify left bottom))
   )
   (label "RELAY_UP+" (at 154.94 157.48 90)
@@
     (pin "2")
   )
+  (symbol (lib_id "Device:C") (at 269.24 86.36 0) (unit 1)
+    (in_bom yes) (on_board yes)
+    (property "Reference" "C13" (id 0) (at 272.161 85.1916 0)
+      (effects (font (size 1.27 1.27)) (justify left))
+    )
+    (property "Value" "100n" (id 1) (at 272.161 87.503 0)
+      (effects (font (size 1.27 1.27)) (justify left))
+    )
+    (property "Footprint" "Capacitor_SMD:C_0603_1608Metric" (id 2) (at 270.2052 90.17 0)
+      (effects (font (size 1.27 1.27)) hide)
+    )
+    (property "Datasheet" "~" (id 3) (at 269.24 86.36 0)
+      (effects (font (size 1.27 1.27)) hide)
+    )
+    (pin "1")
+    (pin "2")
+  )
   (symbol (lib_id "power:+5V") (at 80.01 26.67 270) (unit 1)
     (in_bom yes) (on_board yes) (fields_autoplaced)
@@
       (reference "C12") (unit 1) (value "1uF") (footprint "Capacitor_SMD:C_0603_1608Metric")
     )
+    (path "/b2242582-8a2a-4dd7-9028-8eff339cc1b0"
+      (reference "C13") (unit 1) (value "100n") (footprint "Capacitor_SMD:C_0603_1608Metric")
+    )
     (path "/00000000-0000-0000-0000-000061a495d1"
