File: power-wedge-control.kicad_sch (KiCad schematic)
At the start: 58 parts, among them J1 Conn_01x02, J2 Conn_01x03, J3 Conn_01x02, J4 Conn_01x03, J5 Conn_01x03, J6 Conn_01x06_Female, J7 Conn_01x04_Female, J8 Conn_01x03, J9 MicroSD_Hirose_DM3D-SF, Q1 MMBT3904L, Q2 DMP3099L, Q3 MMBT3904L, Q4 DMP3099L, Q5 MMBT3904L, Q6 MMBT3904L, U1 LM7805_TO220, U3 TLV70233DBV, U4 4050

Commit message: Switch to NC7WZ17P6X buffers for level shifting to SD card.
Parts:
- removed C16: 100n, Capacitor_SMD:C_0603_1608Metric, symbol Device:C
- removed U4: 4050, Package_SO:SOIC-16W_5.3x10.2mm_P1.27mm, symbol 4xxx:4050
- added U5, U6: NC7WZ17P6X, Package_TO_SOT_SMD:SOT-363_SC-70-6, symbol NC7WZ17P6X:NC7WZ17P6X
Connections:
- net +3V3: now also U5.5 (VCC), U6.5 (VCC)
- net CS: now also U5.1 (A1)
- net GND: now also U5.2 (GND), U6.2 (GND)
- net MISO: now also U6.4 (Y2)
- net MOSI: now also U5.3 (A2)
- net SCK: now also U6.1 (A1)
- net SD_CLK: now also U6.6 (Y1)
- net SD_CS: now also U5.6 (Y1)
- net SD_DI: now also U5.4 (Y2)
- net SD_DO: now also U6.3 (A2)
- no-connect marks 45 -> 43
Other:
- moved on the sheet: J9

Commit message: Change 5V regulator LM7805 to LM1117.
Parts:
- removed U1: LM7805_TO220, Package_TO_SOT_THT:TO-220-3_Horizontal_TabDown, symbol Regulator_Linear:LM7805_TO220
- added U1: LM1117-5.0, Package_TO_SOT_SMD:TO-252-2, symbol Regulator_Linear:LM1117-5.0
Connections:
- net +12V: now also U1.3 (VI)
- net +5V: now also U1.2 (VO)
- net GND: now also U1.1 (GND)
Other:
- note added: "Power: 14 mA @ 5V used by each angle sensor (27 mA total)"
Changed lines of the file:
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@@
   (junction (at 33.02 34.29) (diameter 0) (color 0 0 0 0)
   )
+  (junction (at 49.53 34.29) (diameter 0) (color 0 0 0 0)
+  )
   (junction (at 73.66 26.67) (diameter 0) (color 0 0 0 0)
   )
@@
   )
   (junction (at 68.58 172.72) (diameter 0) (color 0 0 0 0)
-  )
-  (junction (at 49.53 34.29) (diameter 0) (color 0 0 0 0)
   )
   (junction (at 172.72 100.33) (diameter 0) (color 0 0 0 0)
@@
     (stroke (width 0) (type default) (color 0 0 0 0))
   )
+  (wire (pts (xy 49.53 34.29) (xy 62.23 34.29))
+    (stroke (width 0) (type default) (color 0 0 0 0))
+  )
   (wire (pts (xy 54.61 165.1) (xy 57.15 165.1))
     (stroke (width 0) (type default) (color 0 0 0 0))
@@
   )
   (wire (pts (xy 95.25 45.72) (xy 107.95 45.72))
-    (stroke (width 0) (type default) (color 0 0 0 0))
-  )
-  (wire (pts (xy 49.53 34.29) (xy 62.23 34.29))
     (stroke (width 0) (type default) (color 0 0 0 0))
   )
@@
   (text "TODO: Do we need 3V3? Or does Huzzah32 Feather make 3.3V?"
     (at 191.77 99.06 0)
+    (effects (font (size 1.27 1.27)) (justify left bottom))
+  )
+  (text "Power: 14 mA @ 5V used by each angle sensor (27 mA total)"
+    (at 19.05 195.58 0)
     (effects (font (size 1.27 1.27)) (justify left bottom))
   )
@@
     (pin "9")
   )
-  (symbol (lib_id "Regulator_Linear:LM7805_TO220") (at 49.53 26.67 0) (unit 1)
-    (in_bom yes) (on_board yes) (fields_autoplaced)
-    (property "Reference" "U1" (id 0) (at 49.53 19.05 0))
-    (property "Value" "LM7805_TO220" (id 1) (at 49.53 21.59 0))
-    (property "Footprint" "Package_TO_SOT_THT:TO-220-3_Horizontal_TabDown" (id 2) (at 49.53 20.955 0)
-      (effects (font (size 1.27 1.27) italic) hide)
-    )
-    (property "Datasheet" "https://www.onsemi.cn/PowerSolutions/document/MC7800-D.PDF" (id 3) (at 49.53 27.94 0)
-      (effects (font (size 1.27 1.27)) hide)
-    )
-    (pin "1")
-    (pin "2")
-    (pin "3")
-  )
   (symbol (lib_id "Jumper:Jumper_2_Bridged") (at 250.19 72.39 0) (unit 1)
     (in_bom yes) (on_board yes)
@@
     (pin "2")
   )
+  (symbol (lib_id "Regulator_Linear:LM1117-5.0") (at 49.53 26.67 0) (unit 1)
+    (in_bom yes) (on_board yes) (fields_autoplaced)
+    (property "Reference" "U1" (id 0) (at 49.53 19.05 0))
+    (property "Value" "LM1117-5.0" (id 1) (at 49.53 21.59 0))
+    (property "Footprint" "Package_TO_SOT_SMD:TO-252-2" (id 2) (at 49.53 26.67 0)
+      (effects (font (size 1.27 1.27)) hide)
+    )
+    (property "Datasheet" "http://www.ti.com/lit/ds/symlink/lm1117.pdf" (id 3) (at 49.53 26.67 0)
+      (effects (font (size 1.27 1.27)) hide)
+    )
+    (pin "1")
+    (pin "2")
+    (pin "3")
+  )
   (symbol (lib_id "Connector:Micro_SD_Card_Det") (at 378.46 33.02 0) (unit 1)
     (in_bom yes) (on_board yes)
@@
       (reference "R20") (unit 1) (value "4k7") (footprint "Resistor_SMD:R_0603_1608Metric")
     )
-    (path "/09a95aec-18d4-4c3a-a99f-ff4812fcae5b"
-      (reference "U1") (unit 1) (value "LM7805_TO220") (footprint "Package_TO_SOT_THT:TO-220-3_Horizontal_TabDown")
+    (path "/a9ad1d23-3e3c-4da7-984e-5168e5db64f1"
+      (reference "U1") (unit 1) (value "LM1117-5.0") (footprint "Package_TO_SOT_SMD:TO-252-2")
     )
     (path "/a2eb388d-0b35-4968-b572-1fb6a3e2fda5/00000000-0000-0000-0000-00005b839616"

Commit message: Flip J3 relay test points away from Uno USB connector.
Connections:
- net EN_RELAY_DN: now also J3.1 (Pin_1); no longer J3.2 (Pin_2)
- net EN_RELAY_UP: now also J3.2 (Pin_2); no longer J3.1 (Pin_1)
Other:
- moved on the sheet: J3
Changed lines of the file:
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@@
     (pin "2")
   )
-  (symbol (lib_id "Connector_Generic:Conn_01x02") (at 109.22 187.96 0) (mirror y) (unit 1)
+  (symbol (lib_id "Connector_Generic:Conn_01x02") (at 109.22 190.5 180) (unit 1)
     (in_bom yes) (on_board yes)
-    (property "Reference" "J3" (id 0) (at 109.22 185.42 0))
+    (property "Reference" "J3" (id 0) (at 109.22 193.04 0))
     (property "Value" "Conn_01x02" (id 1) (at 106.68 189.23 90))
-    (property "Footprint" "Connector_PinHeader_2.54mm:PinHeader_1x02_P2.54mm_Horizontal" (id 2) (at 109.22 187.96 0)
+    (property "Footprint" "Connector_PinHeader_2.54mm:PinHeader_1x02_P2.54mm_Horizontal" (id 2) (at 109.22 190.5 0)
       (effects (font (size 1.27 1.27)) hide)
     )
-    (property "Datasheet" "~" (id 3) (at 109.22 187.96 0)
+    (property "Datasheet" "~" (id 3) (at 109.22 190.5 0)
       (effects (font (size 1.27 1.27)) hide)
     )

Commit message: Change 7SegDisp UI connection pin labels for TLC6C5912.
Connections:
- net CLK renamed RCK
- net LE renamed G
- net OE renamed SER_IN
- net SDI renamed SRCK
Other:
- note added: "TODO: 3V for UI_PWR"
Changed lines of the file:
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@@
+    (effects (font (size 1.27 1.27)) (justify left bottom))
+  )
+  (text "TODO: 3V for UI_PWR" (at 191.77 177.8 0)
     (effects (font (size 1.27 1.27)) (justify left bottom))
   )
@@
     (effects (font (size 1.27 1.27)) (justify left bottom))
   )
+  (label "SRCK" (at 95.25 53.34 0)
+    (effects (font (size 1.27 1.27)) (justify left bottom))
+  )
   (label "MOSI" (at 302.26 27.94 0)
     (effects (font (size 1.27 1.27)) (justify left bottom))
@@
     (effects (font (size 1.27 1.27)) (justify left bottom))
   )
-  (label "CLK" (at 95.25 50.8 0)
-    (effects (font (size 1.27 1.27)) (justify left bottom))
-  )
   (label "EN_OUTPUT" (at 106.68 113.03 0)
     (effects (font (size 1.27 1.27)) (justify left bottom))
@@
     (effects (font (size 1.27 1.27)) (justify left bottom))
   )
+  (label "SER_IN" (at 34.29 121.92 180)
+    (effects (font (size 1.27 1.27)) (justify right bottom))
+  )
   (label "GND" (at 26.67 91.44 0)
     (effects (font (size 1.27 1.27)) (justify left bottom))
@@
     (effects (font (size 1.27 1.27)) (justify left bottom))
   )
-  (label "LE" (at 34.29 124.46 180)
-    (effects (font (size 1.27 1.27)) (justify right bottom))
-  )
   (label "EN_OUTPUT" (at 266.7 67.31 180)
     (effects (font (size 1.27 1.27)) (justify right bottom))
@@
     (effects (font (size 1.27 1.27)) (justify right bottom))
   )
-  (label "CLK" (at 34.29 127 180)
-    (effects (font (size 1.27 1.27)) (justify right bottom))
+  (label "RCK" (at 95.25 50.8 0)
+    (effects (font (size 1.27 1.27)) (justify left bottom))
   )
   (label "SCK" (at 100.33 68.58 0)
     (effects (font (size 1.27 1.27)) (justify left bottom))
   )
-  (label "SDI" (at 34.29 129.54 180)
-    (effects (font (size 1.27 1.27)) (justify right bottom))
+  (label "SER_IN" (at 95.25 45.72 0)
+    (effects (font (size 1.27 1.27)) (justify left bottom))
   )
   (label "SD_CS" (at 346.71 25.4 0)
@@
     (effects (font (size 1.27 1.27)) (justify right bottom))
   )
-  (label "OE" (at 34.29 121.92 180)
+  (label "G" (at 34.29 124.46 180)
     (effects (font (size 1.27 1.27)) (justify right bottom))
   )
@@
     (effects (font (size 1.27 1.27)) (justify right bottom))
   )
+  (label "SRCK" (at 34.29 129.54 180)
+    (effects (font (size 1.27 1.27)) (justify right bottom))
+  )
   (label "EN_RELAY_DN" (at 125.73 193.04 180)
     (effects (font (size 1.27 1.27)) (justify right bottom))
@@
     (effects (font (size 1.27 1.27)) (justify left bottom))
   )
-  (label "LE" (at 95.25 48.26 0)
+  (label "G" (at 95.25 48.26 0)
     (effects (font (size 1.27 1.27)) (justify left bottom))
   )
@@
     (effects (font (size 1.27 1.27)) (justify right bottom))
   )
+  (label "RCK" (at 34.29 127 180)
+    (effects (font (size 1.27 1.27)) (justify right bottom))
+  )
   (label "CS" (at 100.33 60.96 0)
     (effects (font (size 1.27 1.27)) (justify left bottom))
@@
     (effects (font (size 1.27 1.27)) (justify right bottom))
   )
-  (label "SDI" (at 95.25 53.34 0)
-    (effects (font (size 1.27 1.27)) (justify left bottom))
-  )
   (label "SD_CLK" (at 346.71 33.02 0)
     (effects (font (size 1.27 1.27)) (justify left bottom))
@@
     (effects (font (size 1.27 1.27)) (justify left bottom))
   )
-  (label "OE" (at 95.25 45.72 0)
-    (effects (font (size 1.27 1.27)) (justify left bottom))
-  )

Commit message: Move power supply near angle sensors. Swap several MCU pins.
Move button debounce up near MCU pins.
Add top layer zones for thermal at voltage regs.
Connections:
- net +3V3: now also JP2.1 (A)
- net +5V: no longer JP2.1 (A)
- net BTN_DN: now also A1.19 (D4); no longer A1.23 (D8)
- net BTN_UP: now also A1.20 (D5); no longer A1.24 (D9)
- net EN_RELAY_DN: now also A1.17 (D2); no longer A1.18 (D3)
- net EN_RELAY_UP: now also A1.18 (D3); no longer A1.17 (D2)
- net G: now also A1.22 (D7); no longer A1.20 (D5)
- net RCK: now also A1.23 (D8); no longer A1.21 (D6)
- net SER_IN: now also A1.21 (D6); no longer A1.19 (D4)
- net SRCK: now also A1.24 (D9); no longer A1.22 (D7)

Commit message: Add ferrite bead on sensor power.
Parts:
- removed JP4: Jumper_2_Bridged, Jumper:SolderJumper-2_P1.3mm_Bridged_RoundedPad1.0x1.5mm, symbol Jumper:Jumper_2_Bridged
- added L3: 600R/200mA, Inductor_SMD:L_0603_1608Metric, symbol Device:L
Connections:
- net +5V: now also L3.1
- net SENS_PWR: now also L3.2
Changed lines of the file:
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@@
     (stroke (width 0) (type default) (color 0 0 0 0))
   )
-  (wire (pts (xy 241.3 82.55) (xy 245.11 82.55))
+  (wire (pts (xy 241.3 82.55) (xy 246.38 82.55))
     (stroke (width 0) (type default) (color 0 0 0 0))
   )
@@
     (stroke (width 0) (type default) (color 0 0 0 0))
   )
-  (wire (pts (xy 255.27 82.55) (xy 269.24 82.55))
+  (wire (pts (xy 254 82.55) (xy 269.24 82.55))
     (stroke (width 0) (type default) (color 0 0 0 0))
   )
@@
     (pin "2")
   )
+  (symbol (lib_id "Device:L") (at 250.19 82.55 90) (unit 1)
+    (in_bom yes) (on_board yes)
+    (property "Reference" "L3" (id 0) (at 250.19 80.01 90))
+    (property "Value" "600R/200mA" (id 1) (at 250.19 83.82 90))
+    (property "Footprint" "Inductor_SMD:L_0603_1608Metric" (id 2) (at 250.19 82.55 0)
+      (effects (font (size 1.27 1.27)) hide)
+    )
+    (property "Datasheet" "~" (id 3) (at 250.19 82.55 0)
+      (effects (font (size 1.27 1.27)) hide)
+    )
+    (property "SKU" "742792651" (id 4) (at 250.19 82.55 90)
+      (effects (font (size 1.27 1.27)) hide)
+    )
+    (pin "1")
+    (pin "2")
+  )
   (symbol (lib_id "Device:C") (at 106.68 -1.27 0) (unit 1)
     (in_bom yes) (on_board yes)
@@
     (pin "2")
     (pin "3")
-  )
-  (symbol (lib_id "Jumper:Jumper_2_Bridged") (at 250.19 82.55 0) (unit 1)
-    (in_bom yes) (on_board yes)
-    (property "Reference" "JP4" (id 0) (at 250.19 80.01 0))
-    (property "Value" "Jumper_2_Bridged" (id 1) (at 252.73 83.82 0)
-      (effects (font (size 1.27 1.27)) hide)
-    )
-    (property "Footprint" "Jumper:SolderJumper-2_P1.3mm_Bridged_RoundedPad1.0x1.5mm" (id 2) (at 250.19 82.55 0)
-      (effects (font (size 1.27 1.27)) hide)
-    )
-    (property "Datasheet" "~" (id 3) (at 250.19 82.55 0)
-      (effects (font (size 1.27 1.27)) hide)
-    )
-    (pin "1")
-    (pin "2")
   )
   (symbol (lib_id "Connector:Conn_01x04_Female") (at 21.59 91.44 0) (mirror y) (unit 1)
@@
       (reference "JP3") (unit 1) (value "Jumper_2_Bridged") (footprint "Jumper:SolderJumper-2_P1.3mm_Bridged_RoundedPad1.0x1.5mm")
     )
-    (path "/4b796d77-9ca6-4e8c-a34a-6e361ec8087d"
-      (reference "JP4") (unit 1) (value "Jumper_2_Bridged") (footprint "Jumper:SolderJumper-2_P1.3mm_Bridged_RoundedPad1.0x1.5mm")
-    )
     (path "/00000000-0000-0000-0000-000061a99a6f"
       (reference "L1") (unit 1) (value "600R/200mA") (footprint "Inductor_SMD:L_0603_1608Metric")
@@
       (reference "L2") (unit 1) (value "600R/200mA") (footprint "Inductor_SMD:L_0603_1608Metric")
     )
+    (path "/2ef496d7-ab49-4982-9d58-a0c76b781f8d"
+      (reference "L3") (unit 1) (value "600R/200mA") (footprint "Inductor_SMD:L_0603_1608Metric")
+    )
     (path "/b5421a79-02d0-44c8-a2d4-93fa23466e43"

Commit message: Add GND to angle sensor test points.
Parts:
- J8: value Conn_01x03 -> Conn_01x04; footprint Connector_PinHeader_2.54mm:PinHeader_1x03_P2.54mm_Horizontal -> Connector_PinHeader_2.54mm:PinHeader_1x04_P2.54mm_Horizontal; symbol Connector_Generic:Conn_01x03 -> Connector_Generic:Conn_01x04
Connections:
- net GND: now also J8.4 (Pin_4)
Changed lines of the file:
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@@
+    (stroke (width 0) (type default) (color 0 0 0 0))
+  )
+  (wire (pts (xy 114.3 177.8) (xy 128.27 177.8))
     (stroke (width 0) (type default) (color 0 0 0 0))
   )
@@
     (effects (font (size 1.524 1.524)) (justify left bottom))
   )
-  (text "Test point and LED indicators" (at 110.49 181.61 0)
+  (text "Test point and LED indicators" (at 113.03 181.61 0)
     (effects (font (size 1.27 1.27)) (justify left bottom))
   )
@@
   (label "BTN_PWR" (at 24.13 83.82 0)
     (effects (font (size 1.27 1.27)) (justify left bottom))
+  )
+  (label "GND" (at 128.27 177.8 180)
+    (effects (font (size 1.27 1.27)) (justify right bottom))
   )
   (label "EN_OUTPUT" (at 106.68 113.03 0)
@@
     (pin "2")
   )
-  (symbol (lib_id "Connector_Generic:Conn_01x03") (at 109.22 172.72 0) (mirror y) (unit 1)
-    (in_bom yes) (on_board yes)
-    (property "Reference" "J8" (id 0) (at 109.22 170.18 0))
-    (property "Value" "Conn_01x03" (id 1) (at 106.68 173.99 90))
-    (property "Footprint" "Connector_PinHeader_2.54mm:PinHeader_1x03_P2.54mm_Horizontal" (id 2) (at 109.22 172.72 0)
+  (symbol (lib_id "Connector_Generic:Conn_01x04") (at 109.22 172.72 0) (mirror y) (unit 1)
+    (in_bom yes) (on_board yes)
+    (property "Reference" "J8" (id 0) (at 109.22 180.34 0))
+    (property "Value" "Conn_01x04" (id 1) (at 106.68 173.99 90))
+    (property "Footprint" "Connector_PinHeader_2.54mm:PinHeader_1x04_P2.54mm_Horizontal" (id 2) (at 109.22 172.72 0)
       (effects (font (size 1.27 1.27)) hide)
     )
@@
     (pin "2")
     (pin "3")
+    (pin "4")
   )
   (symbol (lib_id "Connector:Conn_01x04_Female") (at 21.59 91.44 0) (mirror y) (unit 1)
@@
     )
     (path "/4525ae04-c30a-4c84-af19-511fb2ef01b1"
-      (reference "J8") (unit 1) (value "Conn_01x03") (footprint "Connector_PinHeader_2.54mm:PinHeader_1x03_P2.54mm_Horizontal")
+      (reference "J8") (unit 1) (value "Conn_01x04") (footprint "Connector_PinHeader_2.54mm:PinHeader_1x04_P2.54mm_Horizontal")
     )
     (path "/aa36bbf1-be88-483c-a548-fa695999538f"

Commit message: WIP. Add support for active-high (15V max) switch input to schematic.
Parts:
- added JP4, JP5: SW_SPDT, Jumper:SolderJumper-3_P2.0mm_Open_TrianglePad1.0x1.5mm, symbol Switch:SW_SPDT
- added Q7, Q8: MMBT3904L, Package_TO_SOT_SMD:SOT-23, symbol Device:Q_NPN_BEC
- added R21, R22: 220k, Resistor_SMD:R_0603_1608Metric, symbol Device:R
- added R23, R24: 10k, Resistor_SMD:R_0603_1608Metric, symbol Device:R
- added U4: 4050, Package_SO:SOIC-16W_5.3x10.2mm_P1.27mm, symbol 4xxx:4050
- U3: footprint SOT-23-5 -> Package_TO_SOT_SMD:SOT-23-5
Connections:
- net BTN_PWR: now also U4.1 (VCC)
- net GND: now also Q7.2 (E), Q8.2 (E), R21.2, R22.2, U4.11, U4.14, U4.5, U4.8 (VSS), U4.9
- net HWDebounce/SW1IN renamed SW1EXT
- net SW1EXT: now also JP4.2 (B)
- net HWDebounce/SW2IN renamed SW2EXT
- net SW2EXT: now also JP5.2 (B)
- new net: Q8.1 (B), R24.1
- new net: R24.2, U4.6
- new net: R23.2, U4.2
- new net: Q7.1 (B), R23.1
- new net SW1IN_15V: JP4.1 (A), R21.1, U4.3
- new net SW2IN_15V: JP5.1 (A), R22.1, U4.7
- new net ~{SW1}: JP4.3 (C), Q7.3 (C)
- new net ~{SW2}: JP5.3 (C), Q8.3 (C)
- no-connect marks 43 -> 47
Other:
- sheet HWDebounce ports: added ~{SW1IN}, ~{SW2IN}; removed SW1IN, SW2IN
- note added: "15V Tolerant HIGH-To-LOW Level Shift (74HC4050)"
- note added: "Inverted, open-collector output"
- note added: "Jumpers to change switch contacts between GND-Open & Active-High"
- note added: "Support Active-High (15V Max) Switch Input"
