File: power-wedge-control.kicad_sch (KiCad schematic)
At the start: 67 parts, among them J1 Conn_01x02, J2 Conn_01x03, J3 Conn_01x02, J4 Conn_01x03, J5 Conn_01x03, J6 Conn_01x06_Female, J7 Conn_01x04_Female, J8 Conn_01x04, J9 MicroSD_Hirose_DM3D-SF, Q1 MMBT3904L, Q2 DMP3099L, Q3 MMBT3904L, Q4 DMP3099L, Q5 MMBT3904L, Q6 MMBT3904L, Q7 MMBT3904L, Q8 MMBT3904L, U1 LM1117-5.0, U3 TLV70233DBV, U4 4050, U5 NC7WZ17P6X, U6 NC7WZ17P6X

Commit message: Switch to optocouplers, remove GND-Open option for up/down switch input.
Parts:
- removed JP4, JP5: SW_SPDT, Jumper:SolderJumper-3_P2.0mm_Open_TrianglePad1.0x1.5mm, symbol Switch:SW_SPDT
- removed Q7, Q8: MMBT3904L, Package_TO_SOT_SMD:SOT-23, symbol Device:Q_NPN_BEC
- removed R23, R24: 10k, Resistor_SMD:R_0603_1608Metric, symbol Device:R
- removed U4: 4050, Package_SO:SOIC-16W_5.3x10.2mm_P1.27mm, symbol 4xxx:4050
- added U4, U7: LTV-817S, Package_DIP:SMDIP-4_W9.53mm, symbol Isolator:LTV-817S
- R21, R22: value 220k -> 1k
Connections:
- net +12V: now also J7.2 (Pin_2), J7.3 (Pin_3)
- net GND: now also U4.2, U4.3, U7.2, U7.3; no longer J7.2 (Pin_2), J7.3 (Pin_3), R21.2, R22.2
- net SW1EXT: now also R21.2
- net SW2EXT: now also R22.2
- net ~{SW1}: now also U4.4
- net ~{SW2}: now also U7.4
- net SW1IN_15V: no longer names the net of R21.1
- net SW1IN_15V: now also U4.1
- net SW2IN_15V: no longer names the net of R22.1
- net SW2IN_15V: now also U7.1
- no-connect marks 47 -> 43
Other:
- note removed: "15V Tolerant HIGH-To-LOW Level Shift (74HC4050)"
- note removed: "Jumpers to change switch contacts between GND-Open & Active-High"

Commit message: Exclude Adafruit Huzzah32 ESP32 from board/bom.
Parts:
- A2: now left out of the parts list
Changed lines of the file:
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@@
   )
   (symbol (lib_id "MCU_Module:Adafruit_Feather_HUZZAH32_ESP32") (at 177.8 50.8 0) (unit 1)
-    (in_bom yes) (on_board yes) (fields_autoplaced)
+    (in_bom no) (on_board no) (fields_autoplaced)
     (property "Reference" "A2" (id 0) (at 179.8194 83.82 0)
       (effects (font (size 1.27 1.27)) (justify left))

Commit message: Add extra test points for mcu pins, power supply rails.
Reduce back ground plane clearance.
Parts:
- added J10: Conn_01x10, Connector_PinHeader_2.54mm:PinHeader_1x10_P2.54mm_Vertical, symbol Connector_Generic:Conn_01x10
- added J11: Conn_01x08, Connector_PinHeader_2.54mm:PinHeader_1x08_P2.54mm_Vertical, symbol Connector_Generic:Conn_01x08
- added J12: Conn_01x06, Connector_PinHeader_2.54mm:PinHeader_1x06_P2.54mm_Vertical, symbol Connector_Generic:Conn_01x06
- added TP1, TP2, TP3: TestPoint, TestPoint:TestPoint_THTPad_D1.5mm_Drill0.7mm, symbol Connector:TestPoint
Connections:
- net +12V: now also TP1.1
- net +3V3: now also TP3.1
- net +5V: now also TP2.1
- net ANGL1_REF5V: now also J12.4 (Pin_4)
- net ANGL2_REF5V: now also J12.3 (Pin_3)
- net BTN_DN: now also J11.5 (Pin_5)
- net BTN_UP: now also J11.6 (Pin_6)
- net CS: now also J10.8 (Pin_8)
- net EN_RELAY_DN: now also J11.3 (Pin_3)
- net EN_RELAY_UP: now also J11.4 (Pin_4)
- net G: now also J11.8 (Pin_8)
- net GND: now also J10.4 (Pin_4)
- net MISO: now also J10.6 (Pin_6)
- net MOSI: now also J10.7 (Pin_7)
- net RCK: now also J10.10 (Pin_10)
- net SCK: now also J10.5 (Pin_5)
- net SER_IN: now also J11.7 (Pin_7)
- net SRCK: now also J10.9 (Pin_9)
- net at A1.10 (A1): now also J12.5 (Pin_5)
- net at A1.13 (SDA/A4): now also J12.2 (Pin_2)
- net at A1.14 (SCL/A5): now also J12.1 (Pin_1)
- net at A1.15 (D0/RX): now also J11.1 (Pin_1)
- net at A1.16 (D1/TX): now also J11.2 (Pin_2)
- net AREF: now reaches A1.30 (AREF)
- net AREF: now also J10.3 (Pin_3)
- net at A1.31 (SDA/A4): now also J10.2 (Pin_2)
- net at A1.32 (SCL/A5): now also J10.1 (Pin_1)
- net at A1.9 (A0): now also J12.6 (Pin_6)
- no-connect marks 43 -> 34

Commit message: Add 100n on 3V3 at sdcard. More clearance near R21. Fix top zone clearances.
Parts:
- added C16: 100n, Capacitor_SMD:C_0603_1608Metric, symbol Device:C
Connections:
- net +3V3: now also C16.1
- net GND: now also C16.2
Changed lines of the file:
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@@
   (junction (at 116.84 3.81) (diameter 0) (color 0 0 0 0)
   )
+  (junction (at 304.8 11.43) (diameter 0) (color 0 0 0 0)
+  )
   (junction (at 172.72 182.88) (diameter 0) (color 0 0 0 0)
+  )
+  (junction (at 304.8 3.81) (diameter 0) (color 0 0 0 0)
   )
   (junction (at 154.94 182.88) (diameter 0) (color 0 0 0 0)
@@
     (stroke (width 0) (type default) (color 0 0 0 0))
   )
+  (wire (pts (xy 304.8 3.81) (xy 309.88 3.81))
+    (stroke (width 0) (type default) (color 0 0 0 0))
+  )
   (wire (pts (xy 139.7 139.7) (xy 137.16 139.7))
     (stroke (width 0) (type default) (color 0 0 0 0))
@@
     (stroke (width 0) (type default) (color 0 0 0 0))
   )
+  (wire (pts (xy 300.99 3.81) (xy 304.8 3.81))
+    (stroke (width 0) (type default) (color 0 0 0 0))
+  )
   (wire (pts (xy 143.51 185.42) (xy 143.51 189.23))
     (stroke (width 0) (type default) (color 0 0 0 0))
@@
     (stroke (width 0) (type default) (color 0 0 0 0))
   )
+  (wire (pts (xy 300.99 11.43) (xy 304.8 11.43))
+    (stroke (width 0) (type default) (color 0 0 0 0))
+  )
   (wire (pts (xy 138.43 80.01) (xy 105.41 80.01))
     (stroke (width 0) (type default) (color 0 0 0 0))
@@
   )
   (wire (pts (xy 102.87 81.28) (xy 102.87 78.74))
+    (stroke (width 0) (type default) (color 0 0 0 0))
+  )
+  (wire (pts (xy 304.8 11.43) (xy 309.88 11.43))
     (stroke (width 0) (type default) (color 0 0 0 0))
   )
@@
     (pin "2")
   )
+  (symbol (lib_id "power:+3V3") (at 300.99 3.81 90) (unit 1)
+    (in_bom yes) (on_board yes)
+    (property "Reference" "#PWR030" (id 0) (at 304.8 3.81 0)
+      (effects (font (size 1.27 1.27)) hide)
+    )
+    (property "Value" "+3V3" (id 1) (at 297.18 3.81 90)
+      (effects (font (size 1.27 1.27)) (justify left))
+    )
+    (property "Footprint" "" (id 2) (at 300.99 3.81 0)
+      (effects (font (size 1.27 1.27)) hide)
+    )
+    (property "Datasheet" "" (id 3) (at 300.99 3.81 0)
+      (effects (font (size 1.27 1.27)) hide)
+    )
+    (pin "1")
+  )
   (symbol (lib_id "Device:C") (at 21.59 30.48 0) (unit 1)
     (in_bom yes) (on_board yes)
@@
     (pin "6")
   )
+  (symbol (lib_id "Device:C") (at 304.8 7.62 0) (unit 1)
+    (in_bom yes) (on_board yes)
+    (property "Reference" "C16" (id 0) (at 307.721 6.4516 0)
+      (effects (font (size 1.27 1.27)) (justify left))
+    )
+    (property "Value" "100n" (id 1) (at 307.721 8.763 0)
+      (effects (font (size 1.27 1.27)) (justify left))
+    )
+    (property "Footprint" "Capacitor_SMD:C_0603_1608Metric" (id 2) (at 305.7652 11.43 0)
+      (effects (font (size 1.27 1.27)) hide)
+    )
+    (property "Datasheet" "~" (id 3) (at 304.8 7.62 0)
+      (effects (font (size 1.27 1.27)) hide)
+    )
+    (pin "1")
+    (pin "2")
+  )
+  (symbol (lib_id "power:GND") (at 300.99 11.43 270) (unit 1)
+    (in_bom yes) (on_board yes)
+    (property "Reference" "#PWR031" (id 0) (at 294.64 11.43 0)
+      (effects (font (size 1.27 1.27)) hide)
+    )
+    (property "Value" "GND" (id 1) (at 297.7388 11.557 90)
+      (effects (font (size 1.27 1.27)) (justify right))
+    )
+    (property "Footprint" "" (id 2) (at 300.99 11.43 0)
+      (effects (font (size 1.27 1.27)) hide)
+    )
+    (property "Datasheet" "" (id 3) (at 300.99 11.43 0)
+      (effects (font (size 1.27 1.27)) hide)
+    )
+    (pin "1")
+  )
   (symbol (lib_id "Device:C") (at 73.66 30.48 0) (unit 1)
     (in_bom yes) (on_board yes)
@@
       (reference "#PWR029") (unit 1) (value "+3V3") (footprint "")
     )
+    (path "/64078d13-213d-4357-8adc-52285fc0747b"
+      (reference "#PWR030") (unit 1) (value "+3V3") (footprint "")
+    )
+    (path "/f99601f5-abdc-494c-aba9-76db1fe40599"
+      (reference "#PWR031") (unit 1) (value "GND") (footprint "")
+    )
     (path "/f2b99750-ca0a-4baf-b958-faf07f4842d2"
       (reference "#PWR0101") (unit 1) (value "+3V3") (footprint "")
@@
       (reference "C15") (unit 1) (value "100n") (footprint "Capacitor_SMD:C_0603_1608Metric")
     )
+    (path "/f98a1b91-9aa3-4c7d-9ab6-cc42f1ef1222"
+      (reference "C16") (unit 1) (value "100n") (footprint "Capacitor_SMD:C_0603_1608Metric")
+    )
     (path "/00000000-0000-0000-0000-000061a495d1"

Commit message: Add hardware manual control option to schematic and WIP layout.
TODO: 4-wires to up/down buttons: +12V, GND, UP input, DN input.
TODO: EN manual to MCU input pin.
TODO: EN manual test/engr pin.
Parts:
- added R23: 200k, Resistor_SMD:R_0603_1608Metric, symbol Device:R
- added SW1: SW_SPST, Connector_PinHeader_2.54mm:PinHeader_1x02_P2.54mm_Horizontal, symbol Switch:SW_SPST
- added U10, U11: 74LVC1G32, Package_TO_SOT_SMD:SOT-23-5, symbol 74xGxx:74LVC1G32
- added U8: SN74LVC08ADRG3, Package_SO:SOIC-14_3.9x8.7mm_P1.27mm, symbol SN74LVC08ADRG3:SN74LVC08ADRG3
- added U9: NC7WZ14P6X, Package_TO_SOT_SMD:SOT-363_SC-70-6, symbol NC7WZ14P6X:NC7WZ14P6X
- J3: footprint Connector_PinHeader_2.54mm:PinHeader_1x02_P2.54mm_Horizontal -> Connector_PinHeader_2.54mm:PinHeader_1x02_P2.54mm_Vertical
Connections:
- net +3V3: now also JP1.1 (A), SW1.2 (B), U10.5 (VCC), U11.5 (VCC), U8.14 (VCC), U9.5 (VCC)
- net +5V: no longer JP1.1 (A)
- net BTN_DN: now also U8.9 (3A)
- net BTN_UP: now also U8.12 (4A)
- net EN_RELAY_DN: now also U10.4; no longer A1.17 (D2), J11.3 (Pin_3)
- net EN_RELAY_UP: now also U11.4; no longer A1.18 (D3), J11.4 (Pin_4)
- net GND: now also R23.1, U10.3 (GND), U11.3 (GND), U8.7 (GND), U9.2 (GND)
- new net: U8.4 (2A), U9.4 (Y2)
- new net: U8.1 (1A), U9.6 (Y1)
- new net: U11.1, U8.11 (4Y)
- new net: U11.2, U8.6 (2Y)
- new net: U10.1, U8.8 (3Y)
- new net: U10.2, U8.3 (1Y)
- new net EN_MANUAL: R23.2, SW1.1 (A), U8.10 (3B), U8.13 (4B), U9.1 (A1), U9.3 (A2)
- new net MCU_RELAY_DN: A1.17 (D2), J11.3 (Pin_3), U8.2 (1B)
- new net MCU_RELAY_UP: A1.18 (D3), J11.4 (Pin_4), U8.5 (2B)
Other:
- note added: "Hardware Manual Control Option"
- note added: "TODO: 4 wires to up/down buttons: +12V, GND, UP input, DN input."
- note added: "TODO: EN manual test/engr pin."
- note added: "TODO: EN manual to MCU input pin."

Commit message: Add test point on manual enable and connect to MCU A1 pin.
Parts:
- added R24: 4k7, Resistor_SMD:R_0603_1608Metric, symbol Device:R
- added TP4: TestPoint, TestPoint:TestPoint_THTPad_D1.5mm_Drill0.7mm, symbol Connector:TestPoint
Connections:
- net EN_MANUAL: now also R24.2, TP4.1
- net at A1.10 (A1), J12.5 (Pin_5): now also R24.1
Changed lines of the file:
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@@
   (junction (at 39.37 248.92) (diameter 0) (color 0 0 0 0)
   )
+  (junction (at 146.05 53.34) (diameter 0) (color 0 0 0 0)
+  )
   (junction (at 172.72 171.45) (diameter 0) (color 0 0 0 0)
   )
@@
   (junction (at 43.18 220.98) (diameter 0) (color 0 0 0 0)
   )
+  (junction (at 146.05 31.75) (diameter 0) (color 0 0 0 0)
+  )
   (junction (at 57.15 184.15) (diameter 0) (color 0 0 0 0)
   )
@@
     (stroke (width 0) (type default) (color 0 0 0 0))
   )
+  (wire (pts (xy 146.05 29.21) (xy 146.05 31.75))
+    (stroke (width 0) (type default) (color 0 0 0 0))
+  )
   (wire (pts (xy 147.32 238.76) (xy 147.32 237.49))
     (stroke (width 0) (type default) (color 0 0 0 0))
@@
     (stroke (width 0) (type default) (color 0 0 0 0))
   )
+  (wire (pts (xy 146.05 31.75) (xy 146.05 40.64))
+    (stroke (width 0) (type default) (color 0 0 0 0))
+  )
   (wire (pts (xy 21.59 26.67) (xy 33.02 26.67))
     (stroke (width 0) (type default) (color 0 0 0 0))
@@
     (stroke (width 0) (type default) (color 0 0 0 0))
   )
+  (wire (pts (xy 146.05 48.26) (xy 146.05 53.34))
+    (stroke (width 0) (type default) (color 0 0 0 0))
+  )
   (wire (pts (xy -49.53 107.95) (xy -34.29 107.95))
     (stroke (width 0) (type default) (color 0 0 0 0))
@@
     (stroke (width 0) (type default) (color 0 0 0 0))
   )
-  (wire (pts (xy 133.35 53.34) (xy 148.59 53.34))
+  (wire (pts (xy 146.05 53.34) (xy 148.59 53.34))
+    (stroke (width 0) (type default) (color 0 0 0 0))
+  )
+  (wire (pts (xy 133.35 53.34) (xy 146.05 53.34))
     (stroke (width 0) (type default) (color 0 0 0 0))
   )
@@
     (effects (font (size 1.27 1.27)) (justify left bottom))
   )
+  (label "EN_MANUAL" (at 146.05 29.21 270)
+    (effects (font (size 1.27 1.27)) (justify right bottom))
+  )
   (label "ANGL2_REF5V" (at 148.59 58.42 180)
     (effects (font (size 1.27 1.27)) (justify right bottom))
@@
     (pin "2")
   )
+  (symbol (lib_id "Device:R") (at 146.05 44.45 180) (unit 1)
+    (in_bom yes) (on_board yes)
+    (property "Reference" "R24" (id 0) (at 148.59 44.45 90))
+    (property "Value" "4k7" (id 1) (at 146.05 44.45 90))
+    (property "Footprint" "Resistor_SMD:R_0603_1608Metric" (id 2) (at 147.828 44.45 90)
+      (effects (font (size 1.27 1.27)) hide)
+    )
+    (property "Datasheet" "" (id 3) (at 146.05 44.45 0))
+    (pin "1")
+    (pin "2")
+  )
   (symbol (lib_id "power:GND") (at 76.2 3.81 270) (unit 1)
     (in_bom yes) (on_board yes)
@@
     (pin "1")
   )
+  (symbol (lib_id "Connector:TestPoint") (at 146.05 31.75 270) (unit 1)
+    (in_bom yes) (on_board yes) (fields_autoplaced)
+    (property "Reference" "TP4" (id 0) (at 151.13 30.4799 90)
+      (effects (font (size 1.27 1.27)) (justify left))
+    )
+    (property "Value" "TestPoint" (id 1) (at 151.13 33.0199 90)
+      (effects (font (size 1.27 1.27)) (justify left))
+    )
+    (property "Footprint" "TestPoint:TestPoint_THTPad_D1.5mm_Drill0.7mm" (id 2) (at 146.05 36.83 0)
+      (effects (font (size 1.27 1.27)) hide)
+    )
+    (property "Datasheet" "~" (id 3) (at 146.05 36.83 0)
+      (effects (font (size 1.27 1.27)) hide)
+    )
+    (pin "1")
+  )
   (symbol (lib_id "power:+12V") (at 118.11 25.4 0) (unit 1)
     (in_bom yes) (on_board yes)
@@
       (reference "R23") (unit 1) (value "200k") (footprint "Resistor_SMD:R_0603_1608Metric")
     )
+    (path "/83c1848e-d5f2-4cfa-8fa9-f41572d92711"
+      (reference "R24") (unit 1) (value "4k7") (footprint "Resistor_SMD:R_0603_1608Metric")
+    )
     (path "/17027fea-91c8-4491-8aaa-146a40ba9ca9"
       (reference "SW1") (unit 1) (value "SW_SPST") (footprint "Connector_PinHeader_2.54mm:PinHeader_1x02_P2.54mm_Horizontal")
@@
       (reference "TP3") (unit 1) (value "TestPoint") (footprint "TestPoint:TestPoint_THTPad_D1.5mm_Drill0.7mm")
     )
+    (path "/c7e381d8-ee41-45c6-90eb-5d8a70d113f4"
+      (reference "TP4") (unit 1) (value "TestPoint") (footprint "TestPoint:TestPoint_THTPad_D1.5mm_Drill0.7mm")
+    )
     (path "/a9ad1d23-3e3c-4da7-984e-5168e5db64f1"

Commit message: 4 wires to up/down buttons: +12V, GND, UP input, DN input.
Move terminal block pin silkscreen labels away from edge.
Connections:
- net +12V: now also J7.4 (Pin_4); no longer J7.2 (Pin_2), J7.3 (Pin_3)
- net GND: now also J7.1 (Pin_1)
- net SW1EXT: now also J7.2 (Pin_2); no longer J7.1 (Pin_1)
- net SW2EXT: now also J7.3 (Pin_3); no longer J7.4 (Pin_4)
Changed lines of the file:
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@@
   (junction (at 106.68 -5.08) (diameter 0) (color 0 0 0 0)
   )
-  (junction (at 26.67 91.44) (diameter 0) (color 0 0 0 0)
-  )
   (junction (at 269.24 82.55) (diameter 0) (color 0 0 0 0)
   )
@@
     (stroke (width 0) (type default) (color 0 0 0 0))
   )
-  (wire (pts (xy 26.67 91.44) (xy 26.67 93.98))
-    (stroke (width 0) (type default) (color 0 0 0 0))
-  )
   (wire (pts (xy 154.94 182.88) (xy 156.21 182.88))
     (stroke (width 0) (type default) (color 0 0 0 0))
@@
     (stroke (width 0) (type default) (color 0 0 0 0))
   )
-  (wire (pts (xy 26.67 88.9) (xy 34.29 88.9))
+  (wire (pts (xy 26.67 91.44) (xy 34.29 91.44))
     (stroke (width 0) (type default) (color 0 0 0 0))
   )
@@
     (stroke (width 0) (type default) (color 0 0 0 0))
   )
-  (wire (pts (xy 26.67 96.52) (xy 34.29 96.52))
+  (wire (pts (xy 26.67 93.98) (xy 34.29 93.98))
     (stroke (width 0) (type default) (color 0 0 0 0))
   )
@@
     (effects (font (size 1.27 1.27)) (justify right bottom))
   )
-  (label "SW1EXT" (at 34.29 88.9 180)
+  (label "SW1EXT" (at 34.29 91.44 180)
     (effects (font (size 1.27 1.27)) (justify right bottom))
   )
@@
     (effects (font (size 1.27 1.27)) (justify right bottom))
   )
-  (label "SW2EXT" (at 34.29 96.52 180)
+  (label "SW2EXT" (at 34.29 93.98 180)
     (effects (font (size 1.27 1.27)) (justify right bottom))
   )
@@
     (pin "9")
   )
+  (symbol (lib_id "power:GND") (at 26.67 88.9 90) (unit 1)
+    (in_bom yes) (on_board yes)
+    (property "Reference" "#PWR0104" (id 0) (at 33.02 88.9 0)
+      (effects (font (size 1.27 1.27)) hide)
+    )
+    (property "Value" "GND" (id 1) (at 29.9212 88.773 90)
+      (effects (font (size 1.27 1.27)) (justify right))
+    )
+    (property "Footprint" "" (id 2) (at 26.67 88.9 0)
+      (effects (font (size 1.27 1.27)) hide)
+    )
+    (property "Datasheet" "" (id 3) (at 26.67 88.9 0)
+      (effects (font (size 1.27 1.27)) hide)
+    )
+    (pin "1")
+  )
   (symbol (lib_id "Device:LED") (at 137.16 193.04 180) (unit 1)
     (in_bom yes) (on_board yes)
@@
     (pin "2")
   )
-  (symbol (lib_id "power:+12V") (at 26.67 91.44 270) (unit 1)
+  (symbol (lib_id "power:+12V") (at 26.67 96.52 270) (unit 1)
     (in_bom yes) (on_board yes)
-    (property "Reference" "#PWR013" (id 0) (at 22.86 91.44 0)
+    (property "Reference" "#PWR013" (id 0) (at 22.86 96.52 0)
       (effects (font (size 1.27 1.27)) hide)
     )
-    (property "Value" "+12V" (id 1) (at 29.9212 91.821 90)
+    (property "Value" "+12V" (id 1) (at 29.9212 96.901 90)
       (effects (font (size 1.27 1.27)) (justify left))
     )
-    (property "Footprint" "" (id 2) (at 26.67 91.44 0)
+    (property "Footprint" "" (id 2) (at 26.67 96.52 0)
       (effects (font (size 1.27 1.27)) hide)
     )
-    (property "Datasheet" "" (id 3) (at 26.67 91.44 0)
+    (property "Datasheet" "" (id 3) (at 26.67 96.52 0)
       (effects (font (size 1.27 1.27)) hide)
     )
@@
       (reference "#PWR0103") (unit 1) (value "+3V3") (footprint "")
     )
+    (path "/7062eec7-b8e2-4710-a6f4-4ecc40a3ed5c"
+      (reference "#PWR0104") (unit 1) (value "GND") (footprint "")
+    )
     (path "/09535cde-9ba2-41fd-bb26-86cd9c93b7a7"
       (reference "A1") (unit 1) (value "Arduino_UNO_R3") (footprint "Module:Arduino_UNO_R3")
@@
       (reference "R23") (unit 1) (value "200k") (footprint "Resistor_SMD:R_0603_1608Metric")
     )
-    (path "/83c1848e-d5f2-4cfa-8fa9-f41572d92711"
+    (path "/83c1848e-d5f2-4cfa-8fa9-f41572d92712"
       (reference "R24") (unit 1) (value "4k7") (footprint "Resistor_SMD:R_0603_1608Metric")
     )

Commit message: Add 470 Ω resistor to limit current on +12V pin to up/down buttons.
Parts:
- added R25: 470, Resistor_SMD:R_0603_1608Metric, symbol Device:R
Connections:
- net +12V: now also R25.1; no longer J7.4 (Pin_4)
- new net: J7.4 (Pin_4), R25.2
Changed lines of the file:
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@@
     (pin "4")
+  )
+  (symbol (lib_id "Device:R") (at 30.48 96.52 270) (unit 1)
+    (in_bom yes) (on_board yes)
+    (property "Reference" "R25" (id 0) (at 30.48 99.06 90))
+    (property "Value" "470" (id 1) (at 30.48 96.52 90))
+    (property "Footprint" "Resistor_SMD:R_0603_1608Metric" (id 2) (at 30.48 94.742 90)
+      (effects (font (size 1.27 1.27)) hide)
+    )
+    (property "Datasheet" "" (id 3) (at 30.48 96.52 0))
+    (pin "1")
+    (pin "2")
   )
   (symbol (lib_id "Connector:Conn_01x04_Female") (at 21.59 91.44 0) (mirror y) (unit 1)
@@
     (pin "2")
   )
-  (symbol (lib_id "power:+12V") (at 26.67 96.52 270) (unit 1)
-    (in_bom yes) (on_board yes)
-    (property "Reference" "#PWR013" (id 0) (at 22.86 96.52 0)
-      (effects (font (size 1.27 1.27)) hide)
-    )
-    (property "Value" "+12V" (id 1) (at 29.9212 96.901 90)
-      (effects (font (size 1.27 1.27)) (justify left))
-    )
-    (property "Footprint" "" (id 2) (at 26.67 96.52 0)
-      (effects (font (size 1.27 1.27)) hide)
-    )
-    (property "Datasheet" "" (id 3) (at 26.67 96.52 0)
+  (symbol (lib_id "power:+12V") (at 34.29 96.52 270) (unit 1)
+    (in_bom yes) (on_board yes)
+    (property "Reference" "#PWR013" (id 0) (at 30.48 96.52 0)
+      (effects (font (size 1.27 1.27)) hide)
+    )
+    (property "Value" "+12V" (id 1) (at 37.5412 96.901 90)
+      (effects (font (size 1.27 1.27)) (justify left))
+    )
+    (property "Footprint" "" (id 2) (at 34.29 96.52 0)
+      (effects (font (size 1.27 1.27)) hide)
+    )
+    (property "Datasheet" "" (id 3) (at 34.29 96.52 0)
       (effects (font (size 1.27 1.27)) hide)
     )
@@
       (reference "R24") (unit 1) (value "4k7") (footprint "Resistor_SMD:R_0603_1608Metric")
     )
+    (path "/4741c2f9-3aad-4ec5-93d7-cfe712a42a5a"
+      (reference "R25") (unit 1) (value "470") (footprint "Resistor_SMD:R_0603_1608Metric")
+    )
     (path "/17027fea-91c8-4491-8aaa-146a40ba9ca9"
